Commit message: add test trolley

File: src/models/models/urdf/test_trolley.urdf.xacro (robot description, xacro)
@@ -4,9 +4,7 @@
     <!--                         Properties (in METERS)                      -->
     <!-- =================================================================== -->
-    <xacro:property name="chassis_width" value="0.4" />
-    <xacro:property name="chassis_length" value="1.5" />
-    <xacro:property name="chassis_height" value="0.2" />
-    <xacro:property name="wheel_diameter" value="0.4318" />
-    <xacro:property name="wheel_thickness" value="0.05" />
+    <xacro:property name="trolley_width" value="0.8" />
+    <xacro:property name="trolley_length" value="1" />
+    <xacro:property name="trolley_height" value="0.05" />
     <xacro:property name="velodyne_diameter" value="0.1" />
     <xacro:property name="velodyne_height" value="0.0869" />
@@ -17,9 +15,6 @@
     <!--                             Materials                               -->
     <!-- =================================================================== -->
-    <material name="chassis">
-        <color rgba="0.93 0.46 0.14 1"/>
-    </material>
-    <material name="wheel">
-        <color rgba="0 0 0 1"/>
+    <material name="trolley">
+        <color rgba="0.54 0.27 0.075 1"/>
     </material>
     <material name="sensor">
@@ -32,35 +27,11 @@
     <link name="base_link">
         <visual>
-            <origin xyz="0 0 ${chassis_height/2}" rpy="0 0 0" />
+            <origin xyz="0 0 ${trolley_height/2}" rpy="0 0 0" />
             <geometry>
-                <box size="${chassis_length} ${chassis_width} ${chassis_height}"/>
+                <box size="${trolley_length} ${trolley_width} ${trolley_height}"/>
             </geometry>
-            <material name="chassis"/>
+            <material name="trolley"/>
         </visual>
     </link>
-    <!-- Wheels -->
-    <xacro:macro name="wheel" params="name side direction">
-        <!-- side is 1, -1 for left, right -->
-        <!-- direction is 1, -1 for front, back -->
-        <link name="${name}_wheel">
-            <visual>
-                <origin xyz="0 0 0" rpy="${pi/2} 0 0" />
-                <geometry>
-                    <cylinder radius="${wheel_diameter/2}" length="${wheel_thickness}"/>
-                </geometry>
-                <material name="wheel"/>
-            </visual>
-        </link>
-        <joint name="${name}_wheel_joint" type="continuous">
-            <axis xyz="0 1 0" rpy="0 0 0" />
-            <parent link="base_link"/>
-            <child link="${name}_wheel"/>
-            <origin xyz="${direction*chassis_length/3} ${side*chassis_width/2 + 0.1*side} ${chassis_height / 2}" rpy="0 0 0"/>
-        </joint>
-    </xacro:macro>
-    <xacro:wheel name="fl" side="1" direction="1"/>
-    <xacro:wheel name="fr" side="-1" direction="1"/>
-    <xacro:wheel name="bl" side="1" direction="-1"/>
-    <xacro:wheel name="br" side="-1" direction="-1"/>
     <!-- Velodyne -->
     <link name="velodyne">
@@ -76,5 +47,5 @@
         <parent link="base_link"/>
         <child link="velodyne"/>
-        <origin xyz="${chassis_length/2 + velodyne_diameter/2} 0 ${velodyne_height/2}" rpy="0 0 0"/>
+        <origin xyz="${trolley_length/2} 0 ${trolley_height + velodyne_height/2}" rpy="0 0 0"/>
     </joint>
     <!-- ZED2i -->
@@ -91,5 +62,5 @@
         <parent link="base_link"/>
         <child link="zed2i"/>
-        <origin xyz="-0.05 0 ${2*chassis_height}" rpy="0 0 0"/>
+        <origin xyz="${-trolley_length/2} 0 ${0.5}" rpy="0 0 0"/>
     </joint>
 </robot>

Commit message: measurements from trolley

File: src/models/models/urdf/test_trolley.urdf.xacro (robot description, xacro)
@@ -4,7 +4,7 @@
     <!--                         Properties (in METERS)                      -->
     <!-- =================================================================== -->
-    <xacro:property name="trolley_width" value="0.8" />
-    <xacro:property name="trolley_length" value="1" />
-    <xacro:property name="trolley_height" value="0.05" />
+    <xacro:property name="trolley_width" value="0.59" />
+    <xacro:property name="trolley_length" value="0.89" />
+    <xacro:property name="trolley_height" value="0.19" />
     <xacro:property name="velodyne_diameter" value="0.1" />
     <xacro:property name="velodyne_height" value="0.0869" />
@@ -47,5 +47,5 @@
         <parent link="base_link"/>
         <child link="velodyne"/>
-        <origin xyz="${trolley_length/2} 0 ${trolley_height + velodyne_height/2}" rpy="0 0 0"/>
+        <origin xyz="${trolley_length/2} 0 ${trolley_height + velodyne_height/2 + 0.02}" rpy="0 0 0"/>
     </joint>
     <!-- ZED2i -->
@@ -62,5 +62,5 @@
         <parent link="base_link"/>
         <child link="zed2i"/>
-        <origin xyz="${-trolley_length/2} 0 ${0.5}" rpy="0 0 0"/>
+        <origin xyz="${-trolley_length/2 + zed2i_length/2} 0 ${0.8 - zed2i_height/2}" rpy="0 0 0"/>
     </joint>
 </robot>

Commit message: zed base link

File: src/models/models/urdf/test_trolley.urdf.xacro (robot description, xacro)
@@ -50,5 +50,5 @@
     </joint>
     <!-- ZED2i -->
-    <link name="zed2i">
+    <link name="zed_base_link">
         <visual>
             <origin xyz="0 0 0" rpy="0 0 0" />
@@ -61,5 +61,5 @@
     <joint name="zed2i_joint" type="fixed">
         <parent link="base_link"/>
-        <child link="zed2i"/>
+        <child link="zed_base_link"/>
         <origin xyz="${-trolley_length/2} 0 ${0.5}" rpy="0 0 0"/>
     </joint>
