Commit message: fiddle with numbers

File: src/models/models/urdf/qev3.urdf.xacro (robot description, xacro)
@@ -7,5 +7,5 @@
     <xacro:property name="chassis_length" value="1.5" />
     <xacro:property name="chassis_height" value="0.2" />
-    <xacro:property name="wheel_diameter" value="0.4318" />
+    <xacro:property name="wheel_diameter" value="0.381" />
     <xacro:property name="wheel_thickness" value="0.05" />
     <xacro:property name="velodyne_diameter" value="0.1" />
@@ -91,5 +91,5 @@
         <parent link="base_link"/>
         <child link="zed2i"/>
-        <origin xyz="-0.05 0 ${2*chassis_height}" rpy="0 0 0"/>
+        <origin xyz="-0.1 0 ${2*chassis_height}" rpy="0 0 0"/>
     </joint>
 </robot>

Commit message: added a transform map to base link

File: src/models/models/urdf/qev3.urdf.xacro (robot description, xacro)
@@ -56,5 +56,5 @@
             <parent link="base_link"/>
             <child link="${name}_wheel"/>
-            <origin xyz="${direction*chassis_length/3} ${side*chassis_width/2 + 0.1*side} ${chassis_height / 2}" rpy="0 0 0"/>
+            <origin xyz="${direction*chassis_length/4} ${side*chassis_width/2 + 0.1*side} ${chassis_height / 4}" rpy="0 0 0"/>
         </joint>
     </xacro:macro>

Commit message: got qev3 dimensions for urdf, new rviz, models start transforms and displays, sim translators publish to model frames

File: src/models/models/urdf/qev3.urdf.xacro (robot description, xacro)
@@ -4,9 +4,9 @@
     <!--                         Properties (in METERS)                      -->
     <!-- =================================================================== -->
-    <xacro:property name="chassis_width" value="0.4" />
-    <xacro:property name="chassis_length" value="1.5" />
-    <xacro:property name="chassis_height" value="0.2" />
+    <xacro:property name="chassis_width" value="0.64" />
+    <xacro:property name="chassis_length" value="2.51" />
+    <xacro:property name="chassis_height" value="0.55" />
     <xacro:property name="wheel_diameter" value="0.381" />
-    <xacro:property name="wheel_thickness" value="0.05" />
+    <xacro:property name="wheel_thickness" value="0.2" />
     <xacro:property name="velodyne_diameter" value="0.1" />
     <xacro:property name="velodyne_height" value="0.0869" />
@@ -32,5 +32,5 @@
     <link name="base_link">
         <visual>
-            <origin xyz="0 0 ${chassis_height/2}" rpy="0 0 0" />
+            <origin xyz="${chassis_length/6} 0 ${chassis_height/6}" rpy="0 0 0" />
             <geometry>
                 <box size="${chassis_length} ${chassis_width} ${chassis_height}"/>
@@ -40,5 +40,5 @@
     </link>
     <!-- Wheels -->
-    <xacro:macro name="wheel" params="name side direction">
+    <xacro:macro name="wheel" params="name loc">
         <!-- side is 1, -1 for left, right -->
         <!-- direction is 1, -1 for front, back -->
@@ -56,11 +56,11 @@
             <parent link="base_link"/>
             <child link="${name}_wheel"/>
-            <origin xyz="${direction*chassis_length/4} ${side*chassis_width/2 + 0.1*side} ${chassis_height / 4}" rpy="0 0 0"/>
+            <origin xyz="${loc}" rpy="0 0 0"/>
         </joint>
     </xacro:macro>
-    <xacro:wheel name="fl" side="1" direction="1"/>
-    <xacro:wheel name="fr" side="-1" direction="1"/>
-    <xacro:wheel name="bl" side="1" direction="-1"/>
-    <xacro:wheel name="br" side="-1" direction="-1"/>
+    <xacro:wheel name="fl" loc="0.67 -0.6 -0.05"/>
+    <xacro:wheel name="fr" loc="0.67 0.6 -0.05"/>
+    <xacro:wheel name="rl" loc="-0.68 -0.6 -0.05"/>
+    <xacro:wheel name="rr" loc="-0.68 0.6 -0.05"/>
     <!-- Velodyne -->
     <link name="velodyne">
@@ -76,5 +76,5 @@
         <parent link="base_link"/>
         <child link="velodyne"/>
-        <origin xyz="${chassis_length/2 + velodyne_diameter/2} 0 ${velodyne_height/2}" rpy="0 0 0"/>
+        <origin xyz="1.65 0 -0.15" rpy="0 0 0"/>
     </joint>
     <!-- ZED2i -->
@@ -91,5 +91,5 @@
         <parent link="base_link"/>
         <child link="zed2i"/>
-        <origin xyz="-0.1 0 ${2*chassis_height}" rpy="0 0 0"/>
+        <origin xyz="-0.1 0 0.6" rpy="0 0 0"/>
     </joint>
 </robot>

Commit message: fixed cam frame

File: src/models/models/urdf/qev3.urdf.xacro (robot description, xacro)
@@ -79,5 +79,5 @@
     </joint>
     <!-- ZED2i -->
-    <link name="zed2i">
+    <link name="zed2i_left_camera_optical_frame">
         <visual>
             <origin xyz="0 0 0" rpy="0 0 0" />
@@ -90,5 +90,5 @@
     <joint name="zed2i_joint" type="fixed">
         <parent link="base_link"/>
-        <child link="zed2i"/>
+        <child link="zed2i_left_camera_optical_frame"/>
         <origin xyz="-0.1 0 0.6" rpy="0 0 0"/>
     </joint>

Commit message: lidar on ground

File: src/models/models/urdf/qev3.urdf.xacro (robot description, xacro)
@@ -76,5 +76,5 @@
         <parent link="base_link"/>
         <child link="velodyne"/>
-        <origin xyz="1.65 0 -0.15" rpy="0 0 0"/>
+        <origin xyz="1.65 0 -0.2" rpy="0 0 0"/>
     </joint>
     <!-- ZED2i -->

Commit message: logging and frame header

File: src/models/models/urdf/qev3.urdf.xacro (robot description, xacro)
@@ -79,5 +79,5 @@
     </joint>
     <!-- ZED2i -->
-    <link name="zed2i_left_camera_optical_frame">
+    <link name="zed2i">
         <visual>
             <origin xyz="0 0 0" rpy="0 0 0" />
@@ -90,5 +90,5 @@
     <joint name="zed2i_joint" type="fixed">
         <parent link="base_link"/>
-        <child link="zed2i_left_camera_optical_frame"/>
+        <child link="zed2i"/>
         <origin xyz="-0.1 0 0.6" rpy="0 0 0"/>
     </joint>

Commit message: for when there isnt a transform published

File: src/models/models/urdf/qev3.urdf.xacro (robot description, xacro)
@@ -93,3 +93,17 @@
         <origin xyz="-0.1 0 0.6" rpy="0 0 0"/>
     </joint>
+    <link name="zed2i_left_camera_optical_frame">
+        <visual>
+            <origin xyz="0 0 0" rpy="0 0 0" />
+            <geometry>
+                <box size="${zed2i_length} ${zed2i_width} ${zed2i_height}"/>
+            </geometry>
+            <material name="sensor"/>
+        </visual>
+    </link>
+    <joint name="frame_joint" type="fixed">
+        <parent link="zed2i"/>
+        <child link="zed2i_left_camera_optical_frame"/>
+        <origin xyz="0 0.05 0" rpy="0 0 0"/>
+    </joint>
 </robot>

Commit message: name changes

File: src/models/models/urdf/qev3.urdf.xacro (robot description, xacro)
@@ -30,5 +30,5 @@
     <!-- =================================================================== -->
     <!-- Base link (chassis) -->
-    <link name="base_link">
+    <link name="car">
         <visual>
             <origin xyz="${chassis_length/6} 0 ${chassis_height/6}" rpy="0 0 0" />
@@ -54,5 +54,5 @@
         <joint name="${name}_wheel_joint" type="continuous">
             <axis xyz="0 1 0" rpy="0 0 0" />
-            <parent link="base_link"/>
+            <parent link="car"/>
             <child link="${name}_wheel"/>
             <origin xyz="${loc}" rpy="0 0 0"/>
@@ -74,5 +74,5 @@
     </link>
     <joint name="velodyne_joint" type="fixed">
-        <parent link="base_link"/>
+        <parent link="car"/>
         <child link="velodyne"/>
         <origin xyz="1.65 0 -0.2" rpy="0 0 0"/>
@@ -89,5 +89,5 @@
     </link>
     <joint name="zed2i_joint" type="fixed">
-        <parent link="base_link"/>
+        <parent link="car"/>
         <child link="zed2i"/>
         <origin xyz="-0.1 0 0.6" rpy="0 0 0"/>
