Commit message: use new lando mesh :)

File: src/common/vehicle_urdf/urdf/qev3.urdf.xacro (robot description, xacro)
@@ -17,7 +17,4 @@
     <!--                             Materials                               -->
     <!-- =================================================================== -->
-    <material name="chassis">
-        <color rgba="0.93 0.46 0.14 1"/>
-    </material>
     <material name="wheel">
         <color rgba="0 0 0 1"/>
@@ -32,7 +29,7 @@
     <link name="car">
         <visual>
-            <origin xyz="${chassis_length/6} 0 ${chassis_height/6}" rpy="0 0 0" />
+            <origin xyz="0 0 0" rpy="0 0 0" />
             <geometry>
-                <box size="${chassis_length} ${chassis_width} ${chassis_height}"/>
+                <mesh filename="file://$(find vehicle_urdf)/meshes/lando.dae"/>
             </geometry>
             <material name="chassis"/>

Commit message: nice visuals for media post, use meshes from EUFS

File: src/common/vehicle_urdf/urdf/qev3.urdf.xacro (robot description, xacro)
@@ -73,5 +73,5 @@
         <parent link="car"/>
         <child link="velodyne"/>
-        <origin xyz="1.65 0 -0.2" rpy="0 0 0"/>
+        <origin xyz="1.590 0 -0.15" rpy="0 0 0"/>
     </joint>
     <!-- ZED2i -->
@@ -88,5 +88,5 @@
         <parent link="car"/>
         <child link="zed2i"/>
-        <origin xyz="-0.1 0 0.6" rpy="0 0 0"/>
+        <origin xyz="-0.370 0 0.900" rpy="0 0 0"/>
     </joint>
     <link name="zed2i_left_camera_optical_frame">

Commit message: fix urdf for cam tf

File: src/common/vehicle_urdf/urdf/qev3.urdf.xacro (robot description, xacro)
@@ -90,17 +90,3 @@
         <origin xyz="-0.370 0 0.900" rpy="0 0 0"/>
     </joint>
-    <link name="zed2i_left_camera_optical_frame">
-        <visual>
-            <origin xyz="0 0 0" rpy="0 0 0" />
-            <geometry>
-                <box size="${zed2i_length} ${zed2i_width} ${zed2i_height}"/>
-            </geometry>
-            <material name="sensor"/>
-        </visual>
-    </link>
-    <joint name="frame_joint" type="fixed">
-        <parent link="zed2i"/>
-        <child link="zed2i_left_camera_optical_frame"/>
-        <origin xyz="0 0.05 0" rpy="0 0 0"/>
-    </joint>
 </robot>

Commit message: i cant stand TFs and these wheels dont move anyway

File: src/common/vehicle_urdf/urdf/qev3.urdf.xacro (robot description, xacro)
@@ -49,5 +49,5 @@
             </visual>
         </link>
-        <joint name="${name}_wheel_joint" type="continuous">
+        <joint name="${name}_wheel_joint" type="fixed">
             <axis xyz="0 1 0" rpy="0 0 0" />
             <parent link="car"/>
