Commit message: visuals and CLI updates

File: src/common/vehicle_urdf/urdf/vehicle.urdf.xacro (robot description, xacro)
@@ -50,5 +50,5 @@
     <xacro:macro name="front_wheel" params="lr_prefix lr_reflect">
       <link name="${lr_prefix}_steering_hinge"/>
-      <joint name="${lr_prefix}_steering_hinge_joint" type="revolute">
+      <joint name="${lr_prefix}_steering_hinge_joint" type="fixed">
         <origin xyz="${wheelbase / 2}
                      ${lr_reflect * ((chassis_width - wheel_width) / 2)}
@@ -60,5 +60,5 @@
         <limit lower="${-1*steering_limit}" upper="${steering_limit}" effort="10000000" velocity="1000000"/>
       </joint>
-      <joint name="front_${lr_prefix}_wheel_joint" type="continuous">
+      <joint name="front_${lr_prefix}_wheel_joint" type="fixed">
         <origin xyz="0 0 0"
                 rpy="0 0 0"/>
@@ -72,5 +72,5 @@
     <!-- Description of how a rear wheel is connected to the chassis -->
     <xacro:macro name="rear_wheel" params="lr_prefix lr_reflect">
-      <joint name="rear_${lr_prefix}_wheel_joint" type="continuous">
+      <joint name="rear_${lr_prefix}_wheel_joint" type="fixed">
         <origin xyz="${-1 * wheelbase / 2}
                      ${lr_reflect * ((chassis_width - wheel_width) / 2)}
