Commit message: condition to change visual for car when we're viewing in operation or afterwards

File: src/common/vehicle_urdf/urdf/qev-3d.urdf.xacro (robot description, xacro)
@@ -3,4 +3,5 @@
   <!--  Get the parameters  -->
   <xacro:arg name="base_frame" default="base_link"/>
+  <xacro:arg name="display_car" default="true"/>
   <xacro:property name="chassis_link" default="chassis"/>
   <xacro:property name="degrees_90" value="1.5708"/>
@@ -15,8 +16,11 @@
     <color rgba="0 0 0 1"/>
   </material>
+  <material name="orange">
+    <color rgba="0.88 0.36 0.035 1"/>
+  </material>
   <!-- Vehicle include -->
   <xacro:include filename="$(find vehicle_urdf)/urdf/vehicle.urdf.xacro"/>
   <!-- Chassis of the car -->
-  <xacro:chassis base_frame="$(arg base_frame)"/>
+  <xacro:chassis base_frame="$(arg base_frame)" display_car="$(arg display_car)"/>
   <!-- Wheels -->
   <xacro:wheels/>

File: src/common/vehicle_urdf/urdf/vehicle.urdf.xacro (robot description, xacro)
@@ -1,5 +1,5 @@
 <?xml version="1.0"?>
 <robot xmlns:xacro="http://www.ros.org/wiki/xacro">
-  <xacro:macro name="chassis" params="base_frame">
+  <xacro:macro name="chassis" params="base_frame display_car">
     <!-- Base Frame -->
     <link name="${base_frame}"/>
@@ -15,8 +15,17 @@
     <link name="${chassis_link}">
       <visual>
-        <origin xyz="0 0 0" rpy="0 0 0"/>
-        <geometry>
-          <mesh filename="file://$(find vehicle_urdf)/meshes/lando.dae"/>
-        </geometry>
+        <xacro:if value="${display_car}">
+          <origin xyz="0 0 0" rpy="0 0 0"/>
+          <geometry>
+            <mesh filename="file://$(find vehicle_urdf)/meshes/lando.dae"/>
+          </geometry>
+        </xacro:if>
+        <xacro:unless value="${display_car}">
+          <origin xyz="0.3 0 0.2" rpy="0 0 0"/>
+          <geometry>
+            <box size="2.5 0.7 0.6"/>
+          </geometry>
+          <material name="orange"/>
+        </xacro:unless>
       </visual>
       <origin xyz="0 0 0" rpy="0 0 0"/>

Commit message: carpark changes 28/8 - lidar working, mapping reliably

File: src/common/vehicle_urdf/urdf/qev-3d.urdf.xacro (robot description, xacro)
@@ -28,8 +28,5 @@
   <xacro:include filename="$(find vehicle_urdf)/urdf/sensors.urdf.xacro"/>
   <xacro:velodyne parent="${chassis_link}" name="velodyne">
-    <origin xyz="1.590 0.0 -0.15" rpy="0 0 0"/>
+    <origin xyz="-0.3 0.0 0.85" rpy="0 0 0"/>
   </xacro:velodyne>
-  <xacro:zed2i parent="${chassis_link}" name="zed2i">
-    <origin xyz="-0.370 0.0 0.900" rpy="0 0 0"/>
-  </xacro:zed2i>
 </robot>

File: src/common/vehicle_urdf/urdf/sensors.urdf.xacro (robot description, xacro)
@@ -35,80 +35,3 @@
     </link>
   </xacro:macro>
-  <material name="zed_mat">
-    <color rgba="0.8 0.8 0.8 0.8"/>
-  </material>
-  <material name="zedm_mat">
-    <color rgba="0 0 0 0.9"/>
-  </material>
-  <material name="zed2_mat">
-    <color rgba="0.25 0.25 0.25 0.99"/>
-  </material>
-  <material name="zed2i_mat">
-    <color rgba="0.25 0.25 0.25 0.99"/>
-  </material>
-  <material name="zedx_mat">
-    <color rgba="0.25 0.25 0.25 0.99"/>
-  </material>
-  <material name="zedxm_mat">
-    <color rgba="0.25 0.25 0.25 0.99"/>
-  </material>
-  <xacro:property name="baseline" value="0.12" />
-  <xacro:property name="height" value="0.03" />
-  <xacro:property name="bottom_slope" value="0.0" />
-  <xacro:property name="screw_offset_x" value="-0.01" />
-  <xacro:property name="screw_offset_z" value="0.0" />
-  <xacro:property name="optical_offset_x" value="-0.01" />
-  <xacro:property name="zed_width" value="0.17525" />
-  <xacro:property name="zed_length" value="0.0373" />
-  <xacro:property name="zed_height" value="0.03025" />
-  <xacro:macro name="zed2i" params="*origin parent name model=zed2i">
-    <!-- Camera mounting point (the threaded screw hole in the bottom) -->
-    <link name="${name}_camera_link" />
-    <joint name="${name}_base_joint" type="fixed">
-      <parent link="${parent}"/>
-      <child link="${name}_camera_link"/>
-      <xacro:insert_block name="origin" />
-    </joint>
-    <!-- Camera Center -->
-    <link name="${name}_camera_center">
-      <visual>
-        <origin xyz="${screw_offset_x} 0 ${screw_offset_z}" rpy="0 0 0"/>
-        <geometry>
-          <box size="${zed_length} ${zed_width} ${zed_height}"/>
-        </geometry>
-        <material name="${model}_mat" />
-      </visual>
-    </link>
-    <joint name="${name}_camera_center_joint" type="fixed">
-      <parent link="${name}_camera_link"/>
-      <child link="${name}_camera_center"/>
-      <origin xyz="0 0 ${height/2}" rpy="0 ${bottom_slope} 0" />
-    </joint>
-    <!-- Left Camera -->
-    <link name="${name}_left_camera_frame" />
-    <joint name="${name}_left_camera_joint" type="fixed">
-      <parent link="${name}_camera_center"/>
-      <child link="${name}_left_camera_frame"/>
-      <origin xyz="${optical_offset_x} ${baseline/2} 0" rpy="0 0 0" />
-    </joint>
-    <link name="${name}_left_camera_optical_frame"/>
-    <joint name="${name}_left_camera_optical_joint" type="fixed">
-      <origin xyz="0 0 0" rpy="-${M_PI/2} 0.0 -${M_PI/2}"/>
-      <parent link="${name}_left_camera_frame"/>
-      <child link="${name}_left_camera_optical_frame"/>
-    </joint>
-    <!-- Right Camera -->
-    <link name="${name}_right_camera_frame" />
-    <joint name="${name}_right_camera_joint" type="fixed">
-      <parent link="${name}_camera_center"/>
-      <child link="${name}_right_camera_frame"/>
-      <origin xyz="${optical_offset_x} -${baseline/2} 0" rpy="0 0 0" />
-    </joint>
-    <link name="${name}_right_camera_optical_frame"/>
-    <joint name="${name}_right_camera_optical_joint" type="fixed">
-      <origin xyz="0 0 0" rpy="-${M_PI/2} 0.0 -${M_PI/2}"/>
-      <parent link="${name}_right_camera_frame"/>
-      <child link="${name}_right_camera_optical_frame"/>
-    </joint>
-  </xacro:macro>
 </robot>

Commit message: new bringup package, configs and urdf changes for ros2_control migration

File: src/common/vehicle_urdf/urdf/qev-3d.urdf.xacro (robot description, xacro)
@@ -19,4 +19,7 @@
     <color rgba="0.88 0.36 0.035 1"/>
   </material>
+  <material name="invisible">
+    <color rgba="0.0 0.0 0.0 0.0"/>
+  </material>
   <!-- Vehicle include -->
   <xacro:include filename="$(find vehicle_urdf)/urdf/vehicle.urdf.xacro"/>
@@ -30,3 +33,5 @@
     <origin xyz="-0.3 0.0 0.85" rpy="0 0 0"/>
   </xacro:velodyne>
+  <!-- ros2_control include -->
+  <xacro:include filename="$(find vehicle_urdf)/urdf/ros2_control.urdf.xacro"/>
 </robot>

File: src/common/vehicle_urdf/urdf/vehicle.urdf.xacro (robot description, xacro)
@@ -35,5 +35,5 @@
   <xacro:macro name="wheels">
     <!-- Wheel description -->
-    <xacro:macro name="wheel" params="lr_prefix fr_prefix">
+    <xacro:macro name="wheel" params="lr_prefix fr_prefix wheel_material:=black">
       <link name="${lr_prefix}_${fr_prefix}_wheel">
         <visual>
@@ -42,5 +42,5 @@
             <cylinder radius="${wheel_diameter / 2}" length="${wheel_width}"/>
           </geometry>
-          <material name="black"/>
+          <material name="${wheel_material}"/>
         </visual>
       </link>
@@ -48,29 +48,55 @@
     <!-- Front and rear wheel descriptions -->
     <!-- Description of how a front wheel is connected to the chassis -->
-    <xacro:macro name="front_wheel" params="lr_prefix lr_reflect">
+    <xacro:macro name="front_wheel" params="lr_prefix lr_reflect wheel_material:=black movable:=false">
       <link name="${lr_prefix}_steering_hinge"/>
-      <joint name="${lr_prefix}_steering_hinge_joint" type="fixed">
-        <origin xyz="${wheelbase / 2}
-                     ${lr_reflect * ((chassis_width - wheel_width) / 2)}
-                     0"
-                rpy="0 0 0"/>
-        <parent link="${chassis_link}"/>
-        <child link="${lr_prefix}_steering_hinge"/>
-        <axis xyz="0 0 1"/>
-        <limit lower="${-1*steering_limit}" upper="${steering_limit}" effort="10000000" velocity="1000000"/>
-      </joint>
-      <joint name="front_${lr_prefix}_wheel_joint" type="fixed">
-        <origin xyz="0 0 0"
-                rpy="0 0 0"/>
-        <parent link="${lr_prefix}_steering_hinge"/>
-        <child link="${lr_prefix}_front_wheel"/>
-        <axis xyz="0 1 0"/>
-        <limit lower="0" upper="0" effort="10000000" velocity="1000000"/>
-      </joint>
-      <xacro:wheel lr_prefix="${lr_prefix}" fr_prefix="front"/>
+      <xacro:if value="${movable}">
+        <joint name="${lr_prefix}_steering_hinge_joint" type="revolute">
+          <origin xyz="${wheelbase / 2}
+                      ${lr_reflect * ((chassis_width - wheel_width) / 2)}
+                      0"
+                  rpy="0 0 0"/>
+          <parent link="${chassis_link}"/>
+          <child link="${lr_prefix}_steering_hinge"/>
+          <axis xyz="0 0 1"/>
+          <limit lower="${-1*steering_limit}" upper="${steering_limit}" effort="10000000" velocity="1000000"/>
+        </joint>
+      </xacro:if>
+      <xacro:unless value="${movable}">
+        <joint name="${lr_prefix}_steering_hinge_joint" type="fixed">
+          <origin xyz="${wheelbase / 2}
+                      ${lr_reflect * ((chassis_width - wheel_width) / 2)}
+                      0"
+                  rpy="0 0 0"/>
+          <parent link="${chassis_link}"/>
+          <child link="${lr_prefix}_steering_hinge"/>
+          <axis xyz="0 0 1"/>
+          <limit lower="${-1*steering_limit}" upper="${steering_limit}" effort="10000000" velocity="1000000"/>
+        </joint>
+      </xacro:unless>
+      <xacro:if value="${movable}">
+        <joint name="front_${lr_prefix}_wheel_joint" type="continuous">
+          <origin xyz="0 0 0"
+                  rpy="0 0 0"/>
+          <parent link="${lr_prefix}_steering_hinge"/>
+          <child link="${lr_prefix}_front_wheel"/>
+          <axis xyz="0 1 0"/>
+          <limit lower="0" upper="0" effort="10000000" velocity="1000000"/>
+        </joint>
+      </xacro:if>
+      <xacro:unless value="${movable}">
+        <joint name="front_${lr_prefix}_wheel_joint" type="fixed">
+          <origin xyz="0 0 0"
+                  rpy="0 0 0"/>
+          <parent link="${lr_prefix}_steering_hinge"/>
+          <child link="${lr_prefix}_front_wheel"/>
+          <axis xyz="0 1 0"/>
+          <limit lower="0" upper="0" effort="10000000" velocity="1000000"/>
+        </joint>
+      </xacro:unless>
+      <xacro:wheel lr_prefix="${lr_prefix}" fr_prefix="front" wheel_material="${wheel_material}"/>
     </xacro:macro>
     <!-- Description of how a rear wheel is connected to the chassis -->
     <xacro:macro name="rear_wheel" params="lr_prefix lr_reflect">
-      <joint name="rear_${lr_prefix}_wheel_joint" type="fixed">
+      <joint name="rear_${lr_prefix}_wheel_joint" type="continuous">
         <origin xyz="${-1 * wheelbase / 2}
                      ${lr_reflect * ((chassis_width - wheel_width) / 2)}
@@ -87,6 +113,8 @@
     <xacro:front_wheel lr_prefix="left" lr_reflect="1"/>
     <xacro:front_wheel lr_prefix="right" lr_reflect="-1"/>
-    <xacro:rear_wheel lr_prefix="left" lr_reflect="1" />
-    <xacro:rear_wheel lr_prefix="right" lr_reflect="-1" />
+    <!-- Virtual front wheel to abstract single steering control -->
+    <xacro:front_wheel lr_prefix="virtual" lr_reflect="0" wheel_material="invisible" movable="true"/>
+    <xacro:rear_wheel lr_prefix="left" lr_reflect="1"/>
+    <xacro:rear_wheel lr_prefix="right" lr_reflect="-1"/>
   </xacro:macro>
 </robot>
