Commit message: Changed map<srting,vector<vector<char>>> to structs and variants when storing topic and interface info

File: src/common/vehicle_urdf/urdf/ros2_control.urdf.xacro (robot description, xacro)
@@ -5,4 +5,5 @@
             <plugin>mock_components/GenericSystem</plugin>
             <param name="calculate_dynamics">true</param>
+            <param name="ackermann_pub_topic">/vehicle/ackermann_cmd</param>
         </hardware>
         <joint name="rear_left_wheel_joint">
@@ -15,4 +16,5 @@
                 <param name="initial_value">0</param>
             </state_interface>
+            <param name="joint_type">driving</param>
         </joint>
         <joint name="rear_right_wheel_joint">
@@ -25,4 +27,20 @@
                 <param name="initial_value">0</param>
             </state_interface>
+            <param name="joint_type">driving</param>
+        </joint>
+        <joint name="rear_virtual_wheel_joint">
+            <command_interface name="acceleration">
+            </command_interface>
+            <state_interface name="position">
+                <param name="initial_value">0</param>
+                <!-- Custom params not implemented in ROS Humble. Co-opting unused param instead -->
+                <param name="data_type">/vehicle/rw_position</param>
+            </state_interface>
+            <state_interface name="velocity">
+                <param name="initial_value">0</param>
+                <!-- Custom params not implemented in ROS Humble. Co-opting unused param instead -->
+                <param name="data_type">/vehicle/velocity</param>
+            </state_interface>
+            <param name="joint_type">driving</param>
         </joint>
         <joint name="virtual_steering_hinge_joint">
@@ -31,5 +49,8 @@
             <state_interface name="position">
                 <param name="initial_value">0</param>
+                <!-- Custom params not implemented in ROS Humble. Co-opting unused param instead -->
+                <param name="data_type">/vehicle/steering_angle</param>
             </state_interface>
+            <param name="joint_type">steering</param>
         </joint>
     </ros2_control>

Commit message: Further config changes for bicycle controller

File: src/common/vehicle_urdf/urdf/ros2_control.urdf.xacro (robot description, xacro)
@@ -3,14 +3,16 @@
     <ros2_control name="qev-3d" type="system">
         <hardware>
-            <plugin>mock_components/GenericSystem</plugin>
-            <param name="calculate_dynamics">true</param>
+            <plugin>qutms_hw_interfaces/Qev3dTopicInterface</plugin>
+            <!-- <plugin>mock_components/GenericSystem</plugin> -->
+            <!-- <param name="calculate_dynamics">true</param> -->
             <param name="ackermann_pub_topic">/vehicle/ackermann_cmd</param>
         </hardware>
-        <joint name="rear_left_wheel_joint">
+        <!-- For Future Tricycle Drive use -->
+        <!-- <joint name="rear_left_wheel_joint">
             <command_interface name="acceleration">
             </command_interface>
-            <!-- <state_interface name="position">
+            <state_interface name="position">
                 <param name="initial_value">0</param>
-            </state_interface> -->
+            </state_interface>
             <state_interface name="velocity">
                 <param name="initial_value">0</param>
@@ -21,12 +23,12 @@
             <command_interface name="acceleration">
             </command_interface>
-            <!-- <state_interface name="position">
+            <state_interface name="position">
                 <param name="initial_value">0</param>
-            </state_interface> -->
+            </state_interface>
             <state_interface name="velocity">
                 <param name="initial_value">0</param>
             </state_interface>
             <param name="joint_type">driving</param>
-        </joint>
+        </joint> -->
         <joint name="rear_virtual_wheel_joint">
             <command_interface name="acceleration">

File: src/common/vehicle_urdf/urdf/vehicle.urdf.xacro (robot description, xacro)
@@ -97,16 +97,30 @@
     </xacro:macro>
     <!-- Description of how a rear wheel is connected to the chassis -->
-    <xacro:macro name="rear_wheel" params="lr_prefix lr_reflect">
-      <joint name="rear_${lr_prefix}_wheel_joint" type="continuous">
-        <origin xyz="${-1 * wheelbase / 2}
-                     ${lr_reflect * ((chassis_width - wheel_width) / 2)}
-                     0"
-                rpy="0 0 0"/>
-        <parent link="${chassis_link}"/>
-        <child link="${lr_prefix}_rear_wheel"/>
-        <axis xyz="0 1 0"/>
-        <limit lower="0" upper="0" effort="10000000" velocity="1000000"/>
-      </joint>
-      <xacro:wheel lr_prefix="${lr_prefix}" fr_prefix="rear"/>
+    <xacro:macro name="rear_wheel" params="lr_prefix lr_reflect wheel_material:=black movable:=false">
+      <xacro:if value="${movable}">
+        <joint name="rear_${lr_prefix}_wheel_joint" type="continuous">
+          <origin xyz="${-1 * wheelbase / 2}
+                      ${lr_reflect * ((chassis_width - wheel_width) / 2)}
+                      0"
+                  rpy="0 0 0"/>
+          <parent link="${chassis_link}"/>
+          <child link="${lr_prefix}_rear_wheel"/>
+          <axis xyz="0 1 0"/>
+          <limit lower="0" upper="0" effort="10000000" velocity="1000000"/>
+        </joint>
+      </xacro:if>
+      <xacro:unless value="${movable}">
+        <joint name="rear_${lr_prefix}_wheel_joint" type="fixed">
+          <origin xyz="${-1 * wheelbase / 2}
+                      ${lr_reflect * ((chassis_width - wheel_width) / 2)}
+                      0"
+                  rpy="0 0 0"/>
+          <parent link="${chassis_link}"/>
+          <child link="${lr_prefix}_rear_wheel"/>
+          <axis xyz="0 1 0"/>
+          <limit lower="0" upper="0" effort="10000000" velocity="1000000"/>
+        </joint>
+      </xacro:unless>
+      <xacro:wheel lr_prefix="${lr_prefix}" fr_prefix="rear" wheel_material="${wheel_material}"/>
     </xacro:macro>
     <!-- Add the wheels -->
@@ -117,4 +131,6 @@
     <xacro:rear_wheel lr_prefix="left" lr_reflect="1"/>
     <xacro:rear_wheel lr_prefix="right" lr_reflect="-1"/>
+    <!-- Virtual rear wheel to abstract single drive control -->
+    <xacro:rear_wheel lr_prefix="virtual" lr_reflect="0" wheel_material="invisible" movable="true"/>
   </xacro:macro>
 </robot>
