Commit message: Update zed2i ros2 driver. new config and link names to match

File: src/common/vehicle_urdf/urdf/sensors.urdf.xacro (robot description, xacro)
@@ -64,8 +64,8 @@
   <xacro:macro name="zed2i" params="*origin parent name model=zed2i">
     <!-- Camera mounting point (the threaded screw hole in the bottom) -->
-    <link name="${name}_base_link" />
+    <link name="${name}_camera_link" />
     <joint name="${name}_base_joint" type="fixed">
       <parent link="${parent}"/>
-      <child link="${name}_base_link"/>
+      <child link="${name}_camera_link"/>
       <xacro:insert_block name="origin" />
     </joint>
@@ -81,5 +81,5 @@
     </link>
     <joint name="${name}_camera_center_joint" type="fixed">
-      <parent link="${name}_base_link"/>
+      <parent link="${name}_camera_link"/>
       <child link="${name}_camera_center"/>
       <origin xyz="0 0 ${height/2}" rpy="0 ${bottom_slope} 0" />

Commit message: Slight changes to EBS code - using global over local

File: src/common/vehicle_urdf/urdf/sensors.urdf.xacro (robot description, xacro)
@@ -3,33 +3,16 @@
   <xacro:macro name="velodyne" params="*origin parent name">
     <!-- base frame to velodyne base -->
-    <joint name="${name}_base_mount_joint" type="fixed">
+      <joint name="${name}_base_mount_joint" type="fixed">
       <xacro:insert_block name="origin" />
       <parent link="${parent}"/>
-      <child link="${name}_base_link"/>
-    </joint>
-    <link name="${name}_base_link">
-      <visual>
-        <geometry>
-          <mesh filename="file://$(find vehicle_urdf)/meshes/VLP16_base_1.dae" />
-        </geometry>
-      </visual>
-      <visual>
-        <geometry>
-          <mesh filename="file://$(find vehicle_urdf)/meshes/VLP16_base_2.dae" />
-        </geometry>
-      </visual>
-    </link>
-    <!-- velodyne base to velodyne scan -->
-    <joint name="${name}_base_scan_joint" type="fixed" >
-      <origin xyz="0 0 0.0377" rpy="0 0 0" />
-      <parent link="${name}_base_link" />
       <child link="${name}"/>
     </joint>
     <link name="${name}">
       <visual>
-        <origin xyz="0 0 -0.0377" />
+        <origin xyz="0 0 0" rpy="0 0 0"/>
         <geometry>
-          <mesh filename="file://$(find vehicle_urdf)/meshes/VLP16_scan.dae" />
+          <cylinder radius="0.0516" length="0.0717"/>
         </geometry>
+        <material name="black"/>
       </visual>
     </link>
