Commit message: urdf, xacro setup

File: src/control/ros2_control/description/qev3d.ros2_control.urdf.xacro (robot description, xacro)
@@ -1,5 +1,5 @@
 <?xml version="1.0"?>
 <robot xmlns:xacro="http://www.ros.org/wiki/xacro">
-  <xacro:macro name="carlikebot_ros2_control" params="name prefix">
+  <xacro:macro name="qev3d_ros2_control" params="name prefix">
     <ros2_control name="${name}" type="system">
       <hardware>

File: src/operations/vehicle_urdf/urdf/qev-3d.urdf.xacro (robot description, xacro)
@@ -1,4 +1,5 @@
 <?xml version="1.0"?>
 <robot name="qev-3d" xmlns:xacro="http://ros.org/wiki/xacro">
+  <xacro:arg name="prefix" default="" />
   <!--  Get the parameters  -->
   <xacro:arg name="base_frame" default="base_link"/>
@@ -19,4 +20,8 @@
     <color rgba="0.88 0.36 0.035 1"/>
   </material>
+  <!-- Import QEV-3D ros2_control description -->
+  <xacro:include filename="$(find src)/control/ros2_control/description/qev3d.ros2_control.urdf.xacro"/>
+  <!-- Declaring wheel joints setup for the controller -->
+  <xacro:qev3d_ros2_control name="QEV3D" prefix="$(arg prefix)" />
   <!-- Vehicle include -->
   <xacro:include filename="$(find vehicle_urdf)/urdf/vehicle.urdf.xacro"/>

Commit message: URDF and xacro update

File: src/control/ros2_control/description/qev3d.ros2_control.urdf.xacro (robot description, xacro)
@@ -1,5 +1,5 @@
 <?xml version="1.0"?>
 <robot xmlns:xacro="http://www.ros.org/wiki/xacro">
-  <xacro:macro name="qev3d_ros2_control" params="name prefix">
+  <xacro:macro name="qev3d_ros2_control" params="name prefix"> <!--Template for the QEV-3D ros2_control description -->
     <ros2_control name="${name}" type="system">
       <hardware>
@@ -8,10 +8,14 @@
         <param name="example_param_hw_stop_duration_sec">3.0</param>
       </hardware>
-      <joint name="${prefix}front_wheel_joint">
+      <joint name="${prefix}virtual_front_wheel_joint">
         <command_interface name="position"/>
+          <param name = "min">-0.28</param>
+          <param name = "max">0.28</param>
         <state_interface name="position"/>
       </joint>
-      <joint name="${prefix}rear_wheel_joint">
+      <joint name="${prefix}virtual_rear_wheel_joint">
         <command_interface name="velocity"/>
+          <param name = "min">-10</param>
+          <param name = "max">10</param>>
         <state_interface name="velocity"/>
         <state_interface name="position"/>

File: src/operations/vehicle_urdf/urdf/vehicle.urdf.xacro (robot description, xacro)
@@ -72,4 +72,10 @@
     <!-- Description of how a rear wheel is connected to the chassis -->
     <xacro:macro name="rear_wheel" params="lr_prefix lr_reflect">
+      <joint name = "virtual_rear_wheel_joint" type = continuous>
+        <origin xyz="0 0 0" rpy="0 0 0"/>
+        <parent link="${chassis_link}"/>
+        <child link="${lr_prefix}_rear_wheel"/>
+        <axis xyz="0 1 0"/>
+      </joint>
       <joint name="rear_${lr_prefix}_wheel_joint" type="fixed">
         <origin xyz="${-1 * wheelbase / 2}
@@ -89,7 +95,6 @@
     <!-- right_front_wheel -->
     <xacro:front_wheel lr_prefix="right" lr_reflect="-1"/>
-    <!-- left_rear_wheel -->
+    <!--  left_rear_wheel -->
     <xacro:rear_wheel lr_prefix="left" lr_reflect="1" />
-    <!-- right_rear_wheel -->
     <xacro:rear_wheel lr_prefix="right" lr_reflect="-1" />
   </xacro:macro>
