Commit message: robot description adjustment for ros2_control

File: src/control/ros2_control/description/qev3d_ros2_control.xacro (robot description, xacro)
@@ -1,6 +1,6 @@
+<?xml version="1.0"?>
 <!-- Copied from the ros2 control Demo code. Change later when hardware is setup -->
-<?xml version="1.0"?>
 <robot xmlns:xacro="http://www.ros.org/wiki/xacro">
-  <xacro:macro name="qev3d_ros2_control" params="name prefix"> <!--Template for the QEV-3D ros2_control description -->
+  <xacro:macro name="qev3d_ros2_control"> <!--Template for the QEV-3D ros2_control description -->
     <ros2_control name="${name}" type="system">
       <hardware>
@@ -9,5 +9,5 @@
         <param name="example_param_hw_stop_duration_sec">3.0</param>
       </hardware>
-      <joint name="${prefix}virtual_front_wheel_joint">
+      <joint name="virtual_front_wheel_joint">
         <command_interface name="position"/>
           <param name = "min">-0.28</param>
@@ -15,5 +15,5 @@
         <state_interface name="position"/>
       </joint>
-      <joint name="${prefix}virtual_rear_wheel_joint">
+      <joint name="virtual_rear_wheel_joint">
         <command_interface name="velocity"/>
           <param name = "min">-10</param>

File: src/operations/vehicle_urdf/urdf/qev-3d.urdf.xacro (robot description, xacro)
@@ -9,5 +9,4 @@
   <xacro:property name="M_PI" value="3.1415926535897931" />
   <xacro:property name="steering_limit" default="0.28"/>
-  <xacro:property name="wheel_diameter" value="0.4064"/>
   <xacro:property name="wheel_width" value="0.2"/>
   <xacro:property name="chassis_width" value="1.6"/>
@@ -23,5 +22,5 @@
   <xacro:include filename="$(find src)/control/ros2_control/description/qev3d.ros2_control.urdf.xacro"/>
   <!-- Declaring wheel joints setup for the controller -->
-  <xacro:qev3d_ros2_control name="QEV3D" prefix="$(arg prefix)" />
+  <xacro:qev3d_ros2_control name="QEV3D" />
   <!-- Vehicle include -->
   <xacro:include filename="$(find vehicle_urdf)/urdf/vehicle.urdf.xacro"/>

File: src/operations/vehicle_urdf/urdf/vehicle.urdf.xacro (robot description, xacro)
@@ -1,4 +1,20 @@
 <?xml version="1.0"?>
 <robot xmlns:xacro="http://www.ros.org/wiki/xacro">
+  <!-- QEV-3D parameters-->
+  <xacro:property name="PI" value="3.1415926535897931"/>
+  <xacro:property name="chassis_width" value="1.6"/>
+  <xacro:property name="wheel_radius" value="0.5"/>
+  <xacro:property name="wheel_width" value="0.2"/>
+  <xacro:property name="wheelbase" value="1.580"/>
+  <xacro:property name="base_height" value="0.3"/>
+  <xacro:property name="base_width" value="0.6"/>
+  <xacro:property name="chassis_link" default="chassis"/>
+  <!--Chassis link name-->
+  <xacro:property name="steering_limit" value="0.28"/>
+  <xacro:property name="degrees_90" value="1.5708"/>
+  <!-- 90 degrees in radians -->
+  <material name="invisible">
+    <color rgba="0 0 0 0"/>
+  </material>
   <xacro:macro name="chassis" params="base_frame display_car">
     <!-- Base Frame -->
@@ -9,5 +25,5 @@
       <child link="${chassis_link}"/>
       <!-- Wheel height off ground -->
-      <origin xyz="0 0 ${wheel_diameter/2}" rpy="0 0 0"/>
+      <origin xyz="0 0 ${wheel_radius}" rpy="0 0 0"/>
       <axis xyz="1 0 0"/>
     </joint>
@@ -33,6 +49,39 @@
   <!-- Wheels -->
   <xacro:macro name="wheels">    <!--Template for the wheels -->
-    <!-- TODO: ADD virtual_front_wheel_joint and virtual_rear_wheel_joint -->
-    <!-- TODO: Remmove the steering_hinge joint and links -->
+    <!-- Virtual wheel for immitation purposes -->
+    <link name="virtual_rear_wheel">
+      <visual>
+        <origin xyz="0 0 0" rpy="${PI/2} 0 ${PI/2}"/>
+        <geometry>
+          <cylinder length="0.01" radius="${wheel_radius}"/>
+        </geometry>
+        <material name="invisible"/>
+      </visual>
+    </link>
+    <link name="virtual_front_wheel">
+      <visual>
+        <origin xyz="0 0 0" rpy="${PI/2} 0 ${PI/2}"/>
+        <geometry>
+          <cylinder length="0.01" radius="${wheel_radius}"/>
+        </geometry>
+        <material name="invisible"/>
+      </visual>
+    </link>
+    <joint name="virtual_rear_wheel_joint" type="continuous">
+      <parent link="${chassis_link}"/>
+      <child link="virtual_rear_wheel"/>
+      <origin xyz="-${wheelbase/2} 0 -${base_height/2}" rpy="0 0 ${PI/2}"/>
+      <axis xyz="1 0 0"/>
+      <limit effort="100.0" velocity="100.0"/>
+      <dynamics damping="0.2"/>
+    </joint>
+    <joint name="virtual_front_wheel_joint" type="revolute">
+      <parent link="${chassis_link}"/>
+      <child link="virtual_front_wheel"/>
+      <origin xyz="${wheelbase/2} 0 -${base_height/2}" rpy="0 0 ${PI/2}"/>
+      <axis xyz="0 0 1"/>
+      <limit lower="-0.4" upper="0.4" effort="100.0" velocity="0.0"/>
+      <dynamics damping="0.2"/>
+    </joint>
     <!-- Wheel visualisation description -->
     <xacro:macro name="wheel" params="lr_prefix fr_prefix">
@@ -41,5 +90,5 @@
           <origin xyz="0 0 0" rpy="${degrees_90} 0 0"/>
           <geometry>
-            <cylinder radius="${wheel_diameter / 2}" length="${wheel_width}"/>
+            <cylinder radius="${wheel_radius}" length="${wheel_width}"/>
           </geometry>
           <material name="black"/>
@@ -57,26 +106,31 @@
                      ${lr_reflect * ((chassis_width - wheel_width) / 2)}
                      0" rpy="0 0 0"/>
-        <parent link="${chassis_link}"/> <!-- connect to the chassis -->
-        <child link="${lr_prefix}_steering_hinge"/> <!-- connect to the steering hinge -->
-        <axis xyz="0 0 1"/> <!-- axis of rotation -->
+        <parent link="${chassis_link}"/>
+        <!-- connect to the chassis -->
+        <child link="${lr_prefix}_steering_hinge"/>
+        <!-- connect to the steering hinge -->
+        <axis xyz="0 0 1"/>
+        <!-- axis of rotation -->
         <limit lower="${-1*steering_limit}" upper="${steering_limit}" effort="10000000" velocity="1000000"/>
       </joint>
       <!-- create a joint connect the {lr}_steering_hinge to the {lr}_front_wheel -->
-      <joint name="front_${lr_prefix}_wheel_joint" type="fixed">
-        <!-- TODO: change type of rear wheel joints to be "revoloute for steering" -->
-        <origin xyz="0 0 0" rpy="0 0 0"/>
-        <parent link="${lr_prefix}_steering_hinge"/> <!-- connect to the {lr} steering hinge -->
-        <child link="${lr_prefix}_front_wheel"/> <!-- connect to the {lr} wheel -->
-        <axis xyz="0 1 0"/> <!-- axis of rotation -->
-        <limit lower="0" upper="0" effort="10000000" velocity="1000000"/>
-        <!-- TODO: add <mimic> to immitate behaviour of virtual_front_wheel_joint -->
+      <joint name="front_${lr_prefix}_wheel_joint" type="revoloute">
+        <!-- connect to the chassis -->
+        <parent link="${chassis_link}"/>
+        <!-- connect to the {lr}_front_wheel -->
+        <child link="${lr_prefix}_front_wheel"/>
+        <origin xyz="-${wheelbase/2} ${base_width/2} -${base_height/2}" rpy="0 0 ${PI/2}"/>
+        <!-- axis of rotation -->
+        <axis xyz="0 0 1"/>
+        <limit lower="-0.4" upper="0.4" effort="1000.0" velocity="0"/>
+        <dynamics damping="0.2"/>
+        <mimic joint="virtual_front_wheel_joint" multiplier="1.0" offset="0.0"/>
       </joint>
-      <!-- launch the macro to add the front wheels pair -->
+      <!-- launch the macro to add the front wheel links pair -->
       <xacro:wheel lr_prefix="${lr_prefix}" fr_prefix="front"/>
     </xacro:macro>
     <!-- Description of how a rear wheel is connected to the chassis -->
     <xacro:macro name="rear_wheel" params="lr_prefix lr_reflect">
-      <joint name="rear_${lr_prefix}_wheel_joint" type="fixed">
-        <!-- TODO: change type of rear wheel joints to be "continuous" for rolling -->
+      <joint name="rear_${lr_prefix}_wheel_joint" type="continuous">
         <origin xyz="${-1 * wheelbase / 2}
                      ${lr_reflect * ((chassis_width - wheel_width) / 2)}
@@ -84,7 +138,8 @@
         <parent link="${chassis_link}"/>
         <child link="${lr_prefix}_rear_wheel"/>
-        <axis xyz="0 1 0"/>
-        <limit lower="0" upper="0" effort="10000000" velocity="1000000"/>
-        <!-- TODO: add <mimic> to immitate behaviour of virtual_rear_wheel_joint -->
+        <axis xyz="1 0 0"/>
+        <dynamics damping="0.2"/>
+        <limit effort="10000000" velocity="1000000"/>
+        <mimic joint="virtual_rear_wheel_joint" multiplier="1.0" offset="0.0"/>
       </joint>
       <!-- Add the wheel -->
