Commit message: Update QEV-3D ROS2 control description and clean up includes

File: src/control/ros2_control/description/qev3d.ros2_control.xacro (robot description, xacro)
@@ -2,5 +2,5 @@
 <!-- Copied from the ros2 control Demo code. Change later when hardware is setup -->
 <robot xmlns:xacro="http://www.ros.org/wiki/xacro">
-  <xacro:macro name="qev3d_ros2_control"> <!--Template for the QEV-3D ros2_control description -->
+  <xacro:macro name="qev3d_ros2_control" params = "name"> <!--Template for the QEV-3D ros2_control description -->
     <ros2_control name="${name}" type="system">
       <hardware>

File: src/operations/vehicle_urdf/urdf/qev-3d.urdf.xacro (robot description, xacro)
@@ -51,5 +51,5 @@
   <!-- ros2_control include -->
   <!-- TODO FIXME: Fix this include path -->
-  <!-- <xacro:include filename="qev3d.ros2_control.xacro"/> -->
-  <!-- <xacro:qev3d_ros2_control name="QEV-3D" /> -->
+  <xacro:include filename="$(find qev3d_ros2_control)/description/qev3d.ros2_control.urdf.xacro"/>
+  <xacro:qev3d_ros2_control name="QEV-3D" />
 </robot>
