Commit message: Refactor URDF files for improved readability and add TODO comments

File: src/operations/vehicle_urdf/urdf/qev-3d.urdf.xacro (robot description, xacro)
@@ -4,6 +4,6 @@
   <!--  Get the parameters  -->
   <xacro:arg name="base_frame" default="base_link"/>
-  <xacro:arg name="display_car" default="true"/>
-  <xacro:property name="chassis_link" default="chassis"/>
+  <xacro:arg name="display_car" default="true"/>  <!--Display the car mesh-->
+  <xacro:property name="chassis_link" default="chassis"/> <!--Chassis link name-->
   <xacro:property name="degrees_90" value="1.5708"/>
   <xacro:property name="M_PI" value="3.1415926535897931" />
@@ -28,5 +28,5 @@
   <!-- Chassis of the car -->
   <xacro:chassis base_frame="$(arg base_frame)" display_car="$(arg display_car)"/>
-  <!-- Wheels -->
+  <!-- Generate the wheels link, joint -->
   <xacro:wheels/>
   <!-- Sensors include -->

File: src/operations/vehicle_urdf/urdf/vehicle.urdf.xacro (robot description, xacro)
@@ -9,6 +9,5 @@
       <child link="${chassis_link}"/>
       <!-- Wheel height off ground -->
-      <origin xyz="0 0 ${wheel_diameter/2}"
-              rpy="0 0 0"/>
+      <origin xyz="0 0 ${wheel_diameter/2}" rpy="0 0 0"/>
       <axis xyz="1 0 0"/>
     </joint>
@@ -33,6 +32,8 @@
   </xacro:macro>
   <!-- Wheels -->
-  <xacro:macro name="wheels">   <!--Template for the wheels -->
-    <!-- Wheel description -->
+  <xacro:macro name="wheels">    <!--Template for the wheels -->
+    <!-- TODO: ADD virtual_front_wheel_joint and virtual_rear_wheel_joint -->
+    <!-- TODO: Remmove the steering_hinge joint and links -->
+    <!-- Wheel visualisation description -->
     <xacro:macro name="wheel" params="lr_prefix fr_prefix">
       <link name="${lr_prefix}_${fr_prefix}_wheel">
@@ -49,24 +50,27 @@
     <!-- Description of how a front wheel is connected to the chassis -->
     <xacro:macro name="front_wheel" params="lr_prefix lr_reflect">
+      <!-- create a link for steering hinge -->
       <link name="${lr_prefix}_steering_hinge"/>
+      <!-- create joint to connect corresponding {lr}_steering_hinge to the chassis -->
       <joint name="${lr_prefix}_steering_hinge_joint" type="fixed">
         <origin xyz="${wheelbase / 2}
                      ${lr_reflect * ((chassis_width - wheel_width) / 2)}
-                     0"
-                rpy="0 0 0"/>
-        <parent link="${chassis_link}"/>
-        <child link="${lr_prefix}_steering_hinge"/>
-        <axis xyz="0 0 1"/>
+                     0" rpy="0 0 0"/>
+        <parent link="${chassis_link}"/> <!-- connect to the chassis -->
+        <child link="${lr_prefix}_steering_hinge"/> <!-- connect to the steering hinge -->
+        <axis xyz="0 0 1"/> <!-- axis of rotation -->
         <limit lower="${-1*steering_limit}" upper="${steering_limit}" effort="10000000" velocity="1000000"/>
       </joint>
+      <!-- create a joint connect the {lr}_steering_hinge to the {lr}_front_wheel -->
       <joint name="front_${lr_prefix}_wheel_joint" type="fixed">
-        <origin xyz="0 0 0"
-                rpy="0 0 0"/>
-        <parent link="${lr_prefix}_steering_hinge"/>
-        <child link="${lr_prefix}_front_wheel"/>
-        <axis xyz="0 1 0"/>
+        <!-- TODO: change type of rear wheel joints to be "revoloute for steering" -->
+        <origin xyz="0 0 0" rpy="0 0 0"/>
+        <parent link="${lr_prefix}_steering_hinge"/> <!-- connect to the {lr} steering hinge -->
+        <child link="${lr_prefix}_front_wheel"/> <!-- connect to the {lr} wheel -->
+        <axis xyz="0 1 0"/> <!-- axis of rotation -->
         <limit lower="0" upper="0" effort="10000000" velocity="1000000"/>
+        <!-- TODO: add <mimic> to immitate behaviour of virtual_front_wheel_joint -->
       </joint>
-      <!-- Add the wheel -->
+      <!-- launch the macro to add the front wheels pair -->
       <xacro:wheel lr_prefix="${lr_prefix}" fr_prefix="front"/>
     </xacro:macro>
@@ -74,13 +78,15 @@
     <xacro:macro name="rear_wheel" params="lr_prefix lr_reflect">
       <joint name="rear_${lr_prefix}_wheel_joint" type="fixed">
+        <!-- TODO: change type of rear wheel joints to be "continuous" for rolling -->
         <origin xyz="${-1 * wheelbase / 2}
                      ${lr_reflect * ((chassis_width - wheel_width) / 2)}
-                     0"
-                rpy="0 0 0"/>
+                     0" rpy="0 0 0"/>
         <parent link="${chassis_link}"/>
         <child link="${lr_prefix}_rear_wheel"/>
         <axis xyz="0 1 0"/>
         <limit lower="0" upper="0" effort="10000000" velocity="1000000"/>
+        <!-- TODO: add <mimic> to immitate behaviour of virtual_rear_wheel_joint -->
       </joint>
+      <!-- Add the wheel -->
       <xacro:wheel lr_prefix="${lr_prefix}" fr_prefix="rear"/>
     </xacro:macro>

Commit message: steering hinge restored and add virtual components

File: src/operations/vehicle_urdf/urdf/qev-3d.urdf.xacro (robot description, xacro)
@@ -1,9 +1,12 @@
 <?xml version="1.0"?>
-<robot name="qev-3d" xmlns:xacro="http://ros.org/wiki/xacro">
+<robot name="qev-3d"
+  xmlns:xacro="http://ros.org/wiki/xacro">
   <xacro:arg name="prefix" default="" />
   <!--  Get the parameters  -->
   <xacro:arg name="base_frame" default="base_link"/>
-  <xacro:arg name="display_car" default="true"/>  <!--Display the car mesh-->
-  <xacro:property name="chassis_link" default="chassis"/> <!--Chassis link name-->
+  <xacro:arg name="display_car" default="true"/>
+  <!--Display the car mesh-->
+  <xacro:property name="chassis_link" default="chassis"/>
+  <!--Chassis link name-->
   <xacro:property name="degrees_90" value="1.5708"/>
   <xacro:property name="M_PI" value="3.1415926535897931" />
@@ -19,8 +22,11 @@
     <color rgba="0.88 0.36 0.035 1"/>
   </material>
+  <material name="invisible">
+    <color rgba="0.0 0.0 0.0 0.0"/>
+  </material>
   <!-- Import QEV-3D ros2_control description -->
   <xacro:include filename="$(find src)/control/ros2_control/description/qev3d.ros2_control.urdf.xacro"/>
   <!-- Declaring wheel joints setup for the controller -->
-  <xacro:qev3d_ros2_control name="QEV3D" />
+  <xacro:qev3d_ros2_control name="QEV-3D" />
   <!-- Vehicle include -->
   <xacro:include filename="$(find vehicle_urdf)/urdf/vehicle.urdf.xacro"/>

File: src/operations/vehicle_urdf/urdf/vehicle.urdf.xacro (robot description, xacro)
@@ -1,20 +1,4 @@
 <?xml version="1.0"?>
 <robot xmlns:xacro="http://www.ros.org/wiki/xacro">
-  <!-- QEV-3D parameters-->
-  <xacro:property name="PI" value="3.1415926535897931"/>
-  <xacro:property name="chassis_width" value="1.6"/>
-  <xacro:property name="wheel_radius" value="0.5"/>
-  <xacro:property name="wheel_width" value="0.2"/>
-  <xacro:property name="wheelbase" value="1.580"/>
-  <xacro:property name="base_height" value="0.3"/>
-  <xacro:property name="base_width" value="0.6"/>
-  <xacro:property name="chassis_link" default="chassis"/>
-  <!--Chassis link name-->
-  <xacro:property name="steering_limit" value="0.28"/>
-  <xacro:property name="degrees_90" value="1.5708"/>
-  <!-- 90 degrees in radians -->
-  <material name="invisible">
-    <color rgba="0 0 0 0"/>
-  </material>
   <xacro:macro name="chassis" params="base_frame display_car">
     <!-- Base Frame -->
@@ -25,5 +9,5 @@
       <child link="${chassis_link}"/>
       <!-- Wheel height off ground -->
-      <origin xyz="0 0 ${wheel_radius}" rpy="0 0 0"/>
+      <origin xyz="0 0 ${wheel_diameter/2}" rpy="0 0 0"/>
       <axis xyz="1 0 0"/>
     </joint>
@@ -48,41 +32,45 @@
   </xacro:macro>
   <!-- Wheels -->
-  <xacro:macro name="wheels">    <!--Template for the wheels -->
+  <xacro:macro name="wheels">
     <!-- Virtual wheel for immitation purposes -->
-    <link name="virtual_rear_wheel">
-      <visual>
-        <origin xyz="0 0 0" rpy="${PI/2} 0 ${PI/2}"/>
-        <geometry>
-          <cylinder length="0.01" radius="${wheel_radius}"/>
-        </geometry>
-        <material name="invisible"/>
-      </visual>
-    </link>
-    <link name="virtual_front_wheel">
-      <visual>
-        <origin xyz="0 0 0" rpy="${PI/2} 0 ${PI/2}"/>
-        <geometry>
-          <cylinder length="0.01" radius="${wheel_radius}"/>
-        </geometry>
-        <material name="invisible"/>
-      </visual>
-    </link>
-    <joint name="virtual_rear_wheel_joint" type="continuous">
-      <parent link="${chassis_link}"/>
-      <child link="virtual_rear_wheel"/>
-      <origin xyz="-${wheelbase/2} 0 -${base_height/2}" rpy="0 0 ${PI/2}"/>
-      <axis xyz="1 0 0"/>
-      <limit effort="100.0" velocity="100.0"/>
-      <dynamics damping="0.2"/>
-    </joint>
-    <joint name="virtual_front_wheel_joint" type="revolute">
-      <parent link="${chassis_link}"/>
-      <child link="virtual_front_wheel"/>
-      <origin xyz="${wheelbase/2} 0 -${base_height/2}" rpy="0 0 ${PI/2}"/>
-      <axis xyz="0 0 1"/>
-      <limit lower="-0.4" upper="0.4" effort="100.0" velocity="0.0"/>
-      <dynamics damping="0.2"/>
-    </joint>
-    <!-- Wheel visualisation description -->
+    <xacro:macro name="virtual_conponents">
+      <link name="virtual_rear_wheel">
+        <visual>
+          <origin xyz="0 0 0" rpy="${PI/2} 0 ${PI/2}"/>
+          <geometry>
+            <cylinder length="0.01" radius="${wheel_radius}"/>
+          </geometry>
+          <material name="invisible"/>
+        </visual>
+      </link>
+      <link name="virtual_front_wheel">
+        <visual>
+          <origin xyz="0 0 0" rpy="${PI/2} 0 ${PI/2}"/>
+          <geometry>
+            <cylinder length="0.01" radius="${wheel_radius}"/>
+          </geometry>
+          <material name="invisible"/>
+        </visual>
+      </link>
+      <joint name="virtual_rear_wheel_joint" type="continuous">
+        <parent link="${chassis_link}"/>
+        <child link="virtual_rear_wheel"/>
+        <origin xyz="-${wheelbase/2} 0 -${base_height/2}" rpy="0 0 ${PI/2}"/>
+        <axis xyz="1 0 0"/>
+        <limit effort="100.0" velocity="100.0"/>
+        <dynamics damping="0.2"/>
+      </joint>
+      <joint name="virtual_front_wheel_joint" type="revolute">
+        <parent link="${chassis_link}"/>
+        <child link="virtual_front_wheel"/>
+        <origin xyz="${wheelbase/2} 0 -${base_height/2}" rpy="0 0 ${PI/2}"/>
+        <axis xyz="0 0 1"/>
+        <limit lower="-0.4" upper="0.4" effort="100.0" velocity="0.0"/>
+        <dynamics damping="0.2"/>
+      </joint>
+    </xacro:macro>
+    <!-- ADDING VIRTUAL COMPONENTS -->
+    <xacro:virtual_conponents/>
+    <!-- Wheel description -->
     <xacro:macro name="wheel" params="lr_prefix fr_prefix">
       <link name="${lr_prefix}_${fr_prefix}_wheel">
@@ -90,5 +78,5 @@
           <origin xyz="0 0 0" rpy="${degrees_90} 0 0"/>
           <geometry>
-            <cylinder radius="${wheel_radius}" length="${wheel_width}"/>
+            <cylinder radius="${wheel_diameter / 2}" length="${wheel_width}"/>
           </geometry>
           <material name="black"/>
@@ -99,7 +87,5 @@
     <!-- Description of how a front wheel is connected to the chassis -->
     <xacro:macro name="front_wheel" params="lr_prefix lr_reflect">
-      <!-- create a link for steering hinge -->
       <link name="${lr_prefix}_steering_hinge"/>
-      <!-- create joint to connect corresponding {lr}_steering_hinge to the chassis -->
       <joint name="${lr_prefix}_steering_hinge_joint" type="fixed">
         <origin xyz="${wheelbase / 2}
@@ -107,30 +93,20 @@
                      0" rpy="0 0 0"/>
         <parent link="${chassis_link}"/>
-        <!-- connect to the chassis -->
         <child link="${lr_prefix}_steering_hinge"/>
-        <!-- connect to the steering hinge -->
         <axis xyz="0 0 1"/>
-        <!-- axis of rotation -->
         <limit lower="${-1*steering_limit}" upper="${steering_limit}" effort="10000000" velocity="1000000"/>
       </joint>
-      <!-- create a joint connect the {lr}_steering_hinge to the {lr}_front_wheel -->
-      <joint name="front_${lr_prefix}_wheel_joint" type="revolute">
-        <!-- connect to the chassis -->
-        <parent link="${chassis_link}"/>
-        <!-- connect to the {lr}_front_wheel -->
+      <joint name="front_${lr_prefix}_wheel_joint" type="fixed">
+        <origin xyz="0 0 0" rpy="0 0 0"/>
+        <parent link="${lr_prefix}_steering_hinge"/>
         <child link="${lr_prefix}_front_wheel"/>
-        <origin xyz="-${wheelbase/2} ${base_width/2} -${base_height/2}" rpy="0 0 ${PI/2}"/>
-        <!-- axis of rotation -->
-        <axis xyz="0 0 1"/>
-        <limit lower="-0.4" upper="0.4" effort="1000.0" velocity="0"/>
-        <dynamics damping="0.2"/>
-        <mimic joint="virtual_front_wheel_joint" multiplier="1.0" offset="0.0"/>
+        <axis xyz="0 1 0"/>
+        <limit lower="0" upper="0" effort="10000000" velocity="1000000"/>
       </joint>
-      <!-- launch the macro to add the front wheel links pair -->
       <xacro:wheel lr_prefix="${lr_prefix}" fr_prefix="front"/>
     </xacro:macro>
     <!-- Description of how a rear wheel is connected to the chassis -->
     <xacro:macro name="rear_wheel" params="lr_prefix lr_reflect">
-      <joint name="rear_${lr_prefix}_wheel_joint" type="continuous">
+      <joint name="rear_${lr_prefix}_wheel_joint" type="fixed">
         <origin xyz="${-1 * wheelbase / 2}
                      ${lr_reflect * ((chassis_width - wheel_width) / 2)}
@@ -138,18 +114,12 @@
         <parent link="${chassis_link}"/>
         <child link="${lr_prefix}_rear_wheel"/>
-        <axis xyz="1 0 0"/>
-        <dynamics damping="0.2"/>
-        <limit effort="10000000" velocity="1000000"/>
-        <mimic joint="virtual_rear_wheel_joint" multiplier="1.0" offset="0.0"/>
+        <axis xyz="0 1 0"/>
+        <limit lower="0" upper="0" effort="10000000" velocity="1000000"/>
       </joint>
-      <!-- Add the wheel -->
       <xacro:wheel lr_prefix="${lr_prefix}" fr_prefix="rear"/>
     </xacro:macro>
     <!-- Add the wheels -->
-    <!-- left_front_wheel -->
     <xacro:front_wheel lr_prefix="left" lr_reflect="1"/>
-    <!-- right_front_wheel -->
     <xacro:front_wheel lr_prefix="right" lr_reflect="-1"/>
-    <!--  left_rear_wheel -->
     <xacro:rear_wheel lr_prefix="left" lr_reflect="1" />
     <xacro:rear_wheel lr_prefix="right" lr_reflect="-1" />

Commit message: virtual joints and links set up

File: src/operations/vehicle_urdf/urdf/qev-3d.urdf.xacro (robot description, xacro)
@@ -9,7 +9,10 @@
   <xacro:property name="chassis_link" default="chassis"/>
   <!--Chassis link name-->
+  <xacro:property name="base_height" value="0.2"/>
   <xacro:property name="degrees_90" value="1.5708"/>
   <xacro:property name="M_PI" value="3.1415926535897931" />
+  <xacro:property name="PI" value="3.1415926535897931" />
   <xacro:property name="steering_limit" default="0.28"/>
+  <xacro:property name="wheel_diameter" value="0.4"/>
   <xacro:property name="wheel_width" value="0.2"/>
   <xacro:property name="chassis_width" value="1.6"/>
@@ -25,8 +28,11 @@
     <color rgba="0.0 0.0 0.0 0.0"/>
   </material>
+  <material name="blue">
+    <color rgba="0.0 0.0 1.0 1.0"/>
+  </material>
   <!-- Import QEV-3D ros2_control description -->
-  <xacro:include filename="$(find src)/control/ros2_control/description/qev3d.ros2_control.urdf.xacro"/>
+  <!-- <xacro:include filename="$(find src)/control/ros2_control/description/qev3d.ros2_control.urdf.xacro"/> -->
   <!-- Declaring wheel joints setup for the controller -->
-  <xacro:qev3d_ros2_control name="QEV-3D" />
+  <!-- <xacro:qev3d_ros2_control name="QEV-3D" /> -->
   <!-- Vehicle include -->
   <xacro:include filename="$(find vehicle_urdf)/urdf/vehicle.urdf.xacro"/>
@@ -41,4 +47,4 @@
   </xacro:velodyne>
   <!-- ros2_control include -->
-  <xacro:include filename="$(find ros2_control)/description/qev3d.ros2_control.urdf.xacro"/>
+  <!-- <xacro:include filename="$(find ros2_control)/description/qev3d.ros2_control.urdf.xacro"/> -->
 </robot>

File: src/operations/vehicle_urdf/urdf/vehicle.urdf.xacro (robot description, xacro)
@@ -39,5 +39,5 @@
           <origin xyz="0 0 0" rpy="${PI/2} 0 ${PI/2}"/>
           <geometry>
-            <cylinder length="0.01" radius="${wheel_radius}"/>
+            <cylinder length="0.01" radius="${wheel_diameter / 2}"/>
           </geometry>
           <material name="invisible"/>
@@ -48,5 +48,5 @@
           <origin xyz="0 0 0" rpy="${PI/2} 0 ${PI/2}"/>
           <geometry>
-            <cylinder length="0.01" radius="${wheel_radius}"/>
+            <cylinder length="0.01" radius="${wheel_diameter / 2}"/>
           </geometry>
           <material name="invisible"/>
@@ -70,6 +70,4 @@
       </joint>
     </xacro:macro>
-    <!-- ADDING VIRTUAL COMPONENTS -->
-    <xacro:virtual_conponents/>
     <!-- Wheel description -->
     <xacro:macro name="wheel" params="lr_prefix fr_prefix">
@@ -88,5 +86,5 @@
     <xacro:macro name="front_wheel" params="lr_prefix lr_reflect">
       <link name="${lr_prefix}_steering_hinge"/>
-      <joint name="${lr_prefix}_steering_hinge_joint" type="fixed">
+      <joint name="${lr_prefix}_steering_hinge_joint" type="revolute">
         <origin xyz="${wheelbase / 2}
                      ${lr_reflect * ((chassis_width - wheel_width) / 2)}
@@ -95,4 +93,5 @@
         <child link="${lr_prefix}_steering_hinge"/>
         <axis xyz="0 0 1"/>
+        <mimic joint="virtual_front_wheel_joint" multiplier="1" offset="0"/>
         <limit lower="${-1*steering_limit}" upper="${steering_limit}" effort="10000000" velocity="1000000"/>
       </joint>
@@ -115,11 +114,21 @@
         <child link="${lr_prefix}_rear_wheel"/>
         <axis xyz="0 1 0"/>
+        <!-- the real rear wheel joint should mimic the behaviour of the continuous virtual rear joint -->
+        <mimic joint="virtual_rear_wheel_joint" multiplier="1" offset="0"/>
         <limit lower="0" upper="0" effort="10000000" velocity="1000000"/>
       </joint>
       <xacro:wheel lr_prefix="${lr_prefix}" fr_prefix="rear"/>
     </xacro:macro>
-    <!-- Add the wheels -->
+    <!-- ADDING VIRTUAL COMPONENTS -->
+    <xacro:virtual_conponents/>
+    <!-- ADD: -->
+    <!-- Links: left_steering_hinge, left_steering_hinge, left_front_wheel, right_front_wheel -->
+    <!-- Joints: right_steering_hinge_joint, left_steering_hinge_joint,  -->
+    <!-- front_left_wheel_joint, front_right_wheel_joint-->
     <xacro:front_wheel lr_prefix="left" lr_reflect="1"/>
     <xacro:front_wheel lr_prefix="right" lr_reflect="-1"/>
+    <!-- ADD: -->
+    <!-- Links: left_rear_wheel, right_rear_wheel -->
+    <!-- Joints: rear_left_wheel_joint, rear_right_wheel_joint,  -->
     <xacro:rear_wheel lr_prefix="left" lr_reflect="1" />
     <xacro:rear_wheel lr_prefix="right" lr_reflect="-1" />

Commit message: change wheels colour to white (too hard to see with black) and change all of fixed joints type ( fixed joints stop the joints from moving).

File: src/operations/vehicle_urdf/urdf/qev-3d.urdf.xacro (robot description, xacro)
@@ -31,4 +31,7 @@
     <color rgba="0.0 0.0 1.0 1.0"/>
   </material>
+  <material name="white">
+    <color rgba="1.0 1.0 1.0 1.0"/>
+  </material>
   <!-- Import QEV-3D ros2_control description -->
   <!-- <xacro:include filename="$(find src)/control/ros2_control/description/qev3d.ros2_control.urdf.xacro"/> -->

File: src/operations/vehicle_urdf/urdf/vehicle.urdf.xacro (robot description, xacro)
@@ -78,5 +78,5 @@
             <cylinder radius="${wheel_diameter / 2}" length="${wheel_width}"/>
           </geometry>
-          <material name="black"/>
+          <material name="white"/>
         </visual>
       </link>
@@ -107,5 +107,5 @@
     <!-- Description of how a rear wheel is connected to the chassis -->
     <xacro:macro name="rear_wheel" params="lr_prefix lr_reflect">
-      <joint name="rear_${lr_prefix}_wheel_joint" type="fixed">
+      <joint name="rear_${lr_prefix}_wheel_joint" type="continuous">
         <origin xyz="${-1 * wheelbase / 2}
                      ${lr_reflect * ((chassis_width - wheel_width) / 2)}

Commit message: Add dummy inertial parameters to vehicle_urdf, added a test urdf file

File: src/operations/vehicle_urdf/urdf/qev-3d.urdf.xacro (robot description, xacro)
@@ -35,8 +35,4 @@
     <color rgba="1.0 1.0 1.0 1.0"/>
   </material>
-  <!-- Import QEV-3D ros2_control description -->
-  <!-- <xacro:include filename="$(find src)/control/ros2_control/description/qev3d.ros2_control.urdf.xacro"/> -->
-  <!-- Declaring wheel joints setup for the controller -->
-  <!-- <xacro:qev3d_ros2_control name="QEV-3D" /> -->
   <!-- Vehicle include -->
   <xacro:include filename="$(find vehicle_urdf)/urdf/vehicle.urdf.xacro"/>

File: src/operations/vehicle_urdf/urdf/vehicle.urdf.xacro (robot description, xacro)
@@ -29,4 +29,9 @@
       </visual>
       <origin xyz="0 0 0" rpy="0 0 0"/>
+      <inertial>
+        <origin xyz="0 0 0" rpy="0 0 0"/>
+        <mass value="1.0"/>
+        <inertia ixx="0.1" ixy="0.0" ixz="0.0" iyy="0.1" iyz="0.0" izz="0.1"/>
+      </inertial>
     </link>
   </xacro:macro>
@@ -43,4 +48,9 @@
           <material name="invisible"/>
         </visual>
+        <inertial>
+          <origin xyz="0 0 0" rpy="0 0 0"/>
+          <mass value="0.1"/>
+          <inertia ixx="0.01" ixy="0.0" ixz="0.0" iyy="0.01" iyz="0.0" izz="0.01"/>
+        </inertial>
       </link>
       <link name="virtual_front_wheel">
@@ -52,4 +62,9 @@
           <material name="invisible"/>
         </visual>
+        <inertial>
+          <origin xyz="0 0 0" rpy="0 0 0"/>
+          <mass value="0.1"/>
+          <inertia ixx="0.01" ixy="0.0" ixz="0.0" iyy="0.01" iyz="0.0" izz="0.01"/>
+        </inertial>
       </link>
       <joint name="virtual_rear_wheel_joint" type="continuous">
@@ -80,4 +95,9 @@
           <material name="white"/>
         </visual>
+        <inertial>
+          <origin xyz="0 0 0" rpy="0 0 0"/>
+          <mass value="0.1"/>
+          <inertia ixx="0.01" ixy="0.0" ixz="0.0" iyy="0.01" iyz="0.0" izz="0.01"/>
+        </inertial>
       </link>
     </xacro:macro>
@@ -85,5 +105,11 @@
     <!-- Description of how a front wheel is connected to the chassis -->
     <xacro:macro name="front_wheel" params="lr_prefix lr_reflect">
-      <link name="${lr_prefix}_steering_hinge"/>
+      <link name="${lr_prefix}_steering_hinge">
+        <inertial>
+          <origin xyz="0 0 0" rpy="0 0 0"/>
+          <mass value="0.1"/>
+          <inertia ixx="0.01" ixy="0.0" ixz="0.0" iyy="0.01" iyz="0.0" izz="0.01"/>
+        </inertial>
+      </link>
       <joint name="${lr_prefix}_steering_hinge_joint" type="revolute">
         <origin xyz="${wheelbase / 2}
