Commit message: Update vehicle bringup dependencies and URDF properties

File: src/operations/vehicle_urdf/urdf/qev-3d.urdf.xacro (robot description, xacro)
@@ -12,4 +12,5 @@
   <xacro:property name="chassis_width" value="1.6"/>
   <xacro:property name="wheelbase" value="1.580"/>
+  <xacro:property name="base_height" value="0.0"/>
   <!-- material -->
   <material name="black">

Commit message: Changes to vehicle_urdf for EUFS_sim compatibility

File: src/operations/vehicle_urdf/urdf/qev-3d.urdf.xacro (robot description, xacro)
@@ -28,5 +28,30 @@
   <xacro:include filename="$(find vehicle_urdf)/urdf/sensors.urdf.xacro"/>
   <xacro:velodyne parent="${chassis_link}" name="velodyne">
-    <origin xyz="-0.3 0.0 0.85" rpy="0 0 0"/>
+    <origin xyz="-0.3 0 1.0532" rpy="0 0 0"/>
   </xacro:velodyne>
+  <gazebo>
+    <plugin
+      filename="libgazebo_ros_race_car.so"
+      name="gazebo_plugins::eufs_plugins::RaceCarPlugin">
+      <command_mode>velocity</command_mode>
+      <wheelbase>1.53</wheelbase>
+      <max_speed>20.0</max_speed>
+      <max_accel>8.0</max_accel>
+      <max_decel>12.0</max_decel>
+      <max_steering_deg>35.0</max_steering_deg>
+      <update_rate>100.0</update_rate>
+      <publish_rate>50.0</publish_rate>
+      <command_timeout>1.0</command_timeout>
+      <map_frame>map</map_frame>
+      <odom_frame>odom</odom_frame>
+      <base_frame>base_link</base_frame>
+      <simulate_transform>false</simulate_transform>
+      <publish_ground_truth>true</publish_ground_truth>
+      <simulate_slam>true</simulate_slam>
+    </plugin>
+    <plugin
+      filename="libgazebo_ros_cone_detection.so"
+      name="gazebo_plugins::eufs_plugins::ConeDetectionPlugin">
+    </plugin>
+  </gazebo>
 </robot>

File: src/operations/vehicle_urdf/urdf/sensors.urdf.xacro (robot description, xacro)
@@ -1,12 +1,19 @@
 <?xml version="1.0"?>
 <robot xmlns:xacro="http://www.ros.org/wiki/xacro">
-  <xacro:macro name="velodyne" params="*origin parent name">
-    <!-- base frame to velodyne base -->
-      <joint name="${name}_base_mount_joint" type="fixed">
-      <xacro:insert_block name="origin" />
+  <xacro:macro name="velodyne" params="*origin parent name enable_lidar:=false enable_laserscan:=false">
+    <joint name="${name}_base_mount_joint" type="fixed">
+      <xacro:insert_block name="origin"/>
       <parent link="${parent}"/>
       <child link="${name}"/>
     </joint>
     <link name="${name}">
+      <inertial>
+        <origin xyz="0 0 0" rpy="0 0 0"/>
+        <mass value="0.1"/>
+        <inertia
+          ixx="0.0001" ixy="0.0" ixz="0.0"
+          iyy="0.0001" iyz="0.0"
+          izz="0.0001"/>
+      </inertial>
       <visual>
         <origin xyz="0 0 0" rpy="0 0 0"/>
@@ -16,5 +23,42 @@
         <material name="black"/>
       </visual>
+      <collision>
+        <origin xyz="0 0 0" rpy="0 0 0"/>
+        <geometry>
+          <cylinder radius="0.0516" length="0.0717"/>
+        </geometry>
+      </collision>
     </link>
+    <gazebo reference="${name}">
+      <sensor name="${name}_gpu_lidar" type="gpu_lidar">
+        <pose>0 0 0 0 0 0</pose>
+        <topic>/lidar</topic>
+        <gz_frame_id>${name}</gz_frame_id>
+        <update_rate>20</update_rate>
+        <always_on>true</always_on>
+        <visualize>true</visualize>
+        <ray>
+          <scan>
+            <horizontal>
+              <samples>240</samples>
+              <resolution>1</resolution>
+              <min_angle>-1</min_angle>
+              <max_angle>1</max_angle>
+            </horizontal>
+            <vertical>
+              <samples>16</samples>
+              <resolution>1</resolution>
+              <min_angle>-0.25</min_angle>
+              <max_angle>0</max_angle>
+            </vertical>
+          </scan>
+          <range>
+            <min>0.3</min>
+            <max>30.0</max>
+            <resolution>0.01</resolution>
+          </range>
+        </ray>
+      </sensor>
+    </gazebo>
   </xacro:macro>
 </robot>

File: src/operations/vehicle_urdf/urdf/vehicle.urdf.xacro (robot description, xacro)
@@ -3,5 +3,14 @@
   <xacro:macro name="chassis" params="base_frame display_car">
     <!-- Base Frame -->
-    <link name="${base_frame}"/>
+    <link name="${base_frame}">
+      <inertial>
+        <origin xyz="0 0 0" rpy="0 0 0"/>
+        <mass value="0.001"/>
+        <inertia
+          ixx="0.000001" ixy="0.0" ixz="0.0"
+          iyy="0.000001" iyz="0.0"
+          izz="0.000001"/>
+      </inertial>
+    </link>
     <!-- Chassis -->
     <joint name="${chassis_link}_joint" type="fixed">
@@ -14,4 +23,18 @@
     </joint>
     <link name="${chassis_link}">
+      <inertial>
+        <origin xyz="0.3 0 0.2" rpy="0 0 0"/>
+        <mass value="300.0"/>
+        <inertia
+          ixx="40.0" ixy="0.0" ixz="0.0"
+          iyy="120.0" iyz="0.0"
+          izz="140.0"/>
+      </inertial>
+      <collision name="chassis_collision">
+        <origin xyz="0.3 0 0.2" rpy="0 0 0"/>
+        <geometry>
+          <box size="2.5 0.7 0.6"/>
+        </geometry>
+      </collision>
       <visual>
         <xacro:if value="${display_car}">
