Commit message: test

File: src/operations/vehicle_urdf/urdf/vehicle.urdf.xacro (robot description, xacro)
@@ -33,5 +33,5 @@
   </xacro:macro>
   <!-- Wheels -->
-  <xacro:macro name="wheels">
+  <xacro:macro name="wheels">   <!--Template for the wheels -->
     <!-- Wheel description -->
     <xacro:macro name="wheel" params="lr_prefix fr_prefix">
@@ -85,7 +85,11 @@
     </xacro:macro>
     <!-- Add the wheels -->
+    <!-- left_front_wheel -->
     <xacro:front_wheel lr_prefix="left" lr_reflect="1"/>
+    <!-- right_front_wheel -->
     <xacro:front_wheel lr_prefix="right" lr_reflect="-1"/>
+    <!-- left_rear_wheel -->
     <xacro:rear_wheel lr_prefix="left" lr_reflect="1" />
+    <!-- right_rear_wheel -->
     <xacro:rear_wheel lr_prefix="right" lr_reflect="-1" />
   </xacro:macro>

Commit message: test

File: src/operations/vehicle_urdf/urdf/vehicle.urdf.xacro (robot description, xacro)
@@ -68,14 +68,9 @@
         <limit lower="0" upper="0" effort="10000000" velocity="1000000"/>
       </joint>
+      <!-- Add the wheel -->
       <xacro:wheel lr_prefix="${lr_prefix}" fr_prefix="front"/>
     </xacro:macro>
     <!-- Description of how a rear wheel is connected to the chassis -->
     <xacro:macro name="rear_wheel" params="lr_prefix lr_reflect">
-      <joint name = "virtual_rear_wheel_joint" type = continuous>
-        <origin xyz="0 0 0" rpy="0 0 0"/>
-        <parent link="${chassis_link}"/>
-        <child link="${lr_prefix}_rear_wheel"/>
-        <axis xyz="0 1 0"/>
-      </joint>
       <joint name="rear_${lr_prefix}_wheel_joint" type="fixed">
         <origin xyz="${-1 * wheelbase / 2}

Commit message: Add launch file for QEV3D vehicle desciption view and fix joint type typo in URDF

File: src/operations/vehicle_urdf/urdf/vehicle.urdf.xacro (robot description, xacro)
@@ -115,5 +115,5 @@
       </joint>
       <!-- create a joint connect the {lr}_steering_hinge to the {lr}_front_wheel -->
-      <joint name="front_${lr_prefix}_wheel_joint" type="revoloute">
+      <joint name="front_${lr_prefix}_wheel_joint" type="revolute">
         <!-- connect to the chassis -->
         <parent link="${chassis_link}"/>

Commit message: car shows up in gazebo now yay

File: src/operations/vehicle_urdf/urdf/vehicle.urdf.xacro (robot description, xacro)
@@ -28,4 +28,10 @@
         </xacro:unless>
       </visual>
+      <collision>
+        <origin xyz="0 0 0" rpy="0 0 0"/>
+        <geometry>
+          <mesh filename="file://$(find vehicle_urdf)/meshes/lando.dae"/>
+        </geometry>
+      </collision>
       <origin xyz="0 0 0" rpy="0 0 0"/>
       <inertial>
@@ -48,4 +54,10 @@
           <material name="invisible"/>
         </visual>
+        <collision>
+          <origin xyz="0 0 0" rpy="${PI/2} 0 ${PI/2}"/>
+          <geometry>
+            <cylinder length="0.01" radius="${wheel_diameter / 2}"/>
+          </geometry>
+        </collision>
         <inertial>
           <origin xyz="0 0 0" rpy="0 0 0"/>
@@ -62,4 +74,10 @@
           <material name="invisible"/>
         </visual>
+        <collision>
+          <origin xyz="0 0 0" rpy="${PI/2} 0 ${PI/2}"/>
+          <geometry>
+            <cylinder length="0.01" radius="${wheel_diameter / 2}"/>
+          </geometry>
+        </collision>
         <inertial>
           <origin xyz="0 0 0" rpy="0 0 0"/>
@@ -95,4 +113,10 @@
           <material name="white"/>
         </visual>
+        <collision>
+          <origin xyz="0 0 0" rpy="${degrees_90} 0 0"/>
+          <geometry>
+            <cylinder radius="${wheel_diameter / 2}" length="${wheel_width}"/>
+          </geometry>
+        </collision>
         <inertial>
           <origin xyz="0 0 0" rpy="0 0 0"/>

Commit message: Add qev_controllers configuration and description files for ROS2 control

File: src/operations/vehicle_urdf/urdf/vehicle.urdf.xacro (robot description, xacro)
@@ -1,4 +1,5 @@
 <?xml version="1.0"?>
 <robot xmlns:xacro="http://www.ros.org/wiki/xacro">
+  <xacro:property name="M_PI" value="3.14159265359"/>
   <xacro:macro name="chassis" params="base_frame display_car">
     <!-- Base Frame -->
@@ -9,6 +10,5 @@
       <child link="${chassis_link}"/>
       <!-- Wheel height off ground -->
-      <origin xyz="0 0 ${wheel_diameter/2}"
-              rpy="0 0 0"/>
+      <origin xyz="0 0 ${wheel_diameter/2}" rpy="0 0 0"/>
       <axis xyz="1 0 0"/>
     </joint>
@@ -34,4 +34,41 @@
   <!-- Wheels -->
   <xacro:macro name="wheels">
+    <!-- Virtual wheel for immitation purposes -->
+    <xacro:macro name="virtual_conponents">
+      <link name="virtual_rear_wheel">
+        <visual>
+          <origin xyz="0 0 0" rpy="${M_PI/2} 0 ${M_PI/2}"/>
+          <geometry>
+            <cylinder length="0.01" radius="${wheel_diameter / 2}"/>
+          </geometry>
+          <material name="invisible"/>
+        </visual>
+      </link>
+      <link name="virtual_front_wheel">
+        <visual>
+          <origin xyz="0 0 0" rpy="${M_PI/2} 0 ${M_PI/2}"/>
+          <geometry>
+            <cylinder length="0.01" radius="${wheel_diameter / 2}"/>
+          </geometry>
+          <material name="invisible"/>
+        </visual>
+      </link>
+      <joint name="virtual_rear_wheel_joint" type="continuous">
+        <parent link="${chassis_link}"/>
+        <child link="virtual_rear_wheel"/>
+        <origin xyz="-${wheelbase/2} 0 -${base_height/2}" rpy="0 0 ${M_PI/2}"/>
+        <axis xyz="1 0 0"/>
+        <limit effort="100.0" velocity="100.0"/>
+        <dynamics damM_PIng="0.2"/>
+      </joint>
+      <joint name="virtual_front_wheel_joint" type="revolute">
+        <parent link="${chassis_link}"/>
+        <child link="virtual_front_wheel"/>
+        <origin xyz="${wheelbase/2} 0 -${base_height/2}" rpy="0 0 ${M_PI/2}"/>
+        <axis xyz="0 0 1"/>
+        <limit lower="-0.4" upper="0.4" effort="100.0" velocity="0.0"/>
+        <dynamics damM_PIng="0.2"/>
+      </joint>
+    </xacro:macro>
     <!-- Wheel description -->
     <xacro:macro name="wheel" params="lr_prefix fr_prefix">
@@ -42,5 +79,5 @@
             <cylinder radius="${wheel_diameter / 2}" length="${wheel_width}"/>
           </geometry>
-          <material name="black"/>
+          <material name="white"/>
         </visual>
       </link>
@@ -50,17 +87,16 @@
     <xacro:macro name="front_wheel" params="lr_prefix lr_reflect">
       <link name="${lr_prefix}_steering_hinge"/>
-      <joint name="${lr_prefix}_steering_hinge_joint" type="fixed">
+      <joint name="${lr_prefix}_steering_hinge_joint" type="revolute">
         <origin xyz="${wheelbase / 2}
                      ${lr_reflect * ((chassis_width - wheel_width) / 2)}
-                     0"
-                rpy="0 0 0"/>
+                     0" rpy="0 0 0"/>
         <parent link="${chassis_link}"/>
         <child link="${lr_prefix}_steering_hinge"/>
         <axis xyz="0 0 1"/>
+        <mimic joint="virtual_front_wheel_joint" multiplier="1" offset="0"/>
         <limit lower="${-1*steering_limit}" upper="${steering_limit}" effort="10000000" velocity="1000000"/>
       </joint>
       <joint name="front_${lr_prefix}_wheel_joint" type="fixed">
-        <origin xyz="0 0 0"
-                rpy="0 0 0"/>
+        <origin xyz="0 0 0" rpy="0 0 0"/>
         <parent link="${lr_prefix}_steering_hinge"/>
         <child link="${lr_prefix}_front_wheel"/>
@@ -72,19 +108,28 @@
     <!-- Description of how a rear wheel is connected to the chassis -->
     <xacro:macro name="rear_wheel" params="lr_prefix lr_reflect">
-      <joint name="rear_${lr_prefix}_wheel_joint" type="fixed">
+      <joint name="rear_${lr_prefix}_wheel_joint" type="continuous">
         <origin xyz="${-1 * wheelbase / 2}
                      ${lr_reflect * ((chassis_width - wheel_width) / 2)}
-                     0"
-                rpy="0 0 0"/>
+                     0" rpy="0 0 0"/>
         <parent link="${chassis_link}"/>
         <child link="${lr_prefix}_rear_wheel"/>
         <axis xyz="0 1 0"/>
+        <!-- the real rear wheel joint should mimic the behaviour of the continuous virtual rear joint -->
+        <mimic joint="virtual_rear_wheel_joint" multiplier="1" offset="0"/>
         <limit lower="0" upper="0" effort="10000000" velocity="1000000"/>
       </joint>
       <xacro:wheel lr_prefix="${lr_prefix}" fr_prefix="rear"/>
     </xacro:macro>
-    <!-- Add the wheels -->
+    <!-- ADDING VIRTUAL COMPONENTS -->
+    <xacro:virtual_conponents/>
+    <!-- ADD: -->
+    <!-- Links: left_steering_hinge, left_steering_hinge, left_front_wheel, right_front_wheel -->
+    <!-- Joints: right_steering_hinge_joint, left_steering_hinge_joint,  -->
+    <!-- front_left_wheel_joint, front_right_wheel_joint-->
     <xacro:front_wheel lr_prefix="left" lr_reflect="1"/>
     <xacro:front_wheel lr_prefix="right" lr_reflect="-1"/>
+    <!-- ADD: -->
+    <!-- Links: left_rear_wheel, right_rear_wheel -->
+    <!-- Joints: rear_left_wheel_joint, rear_right_wheel_joint,  -->
     <xacro:rear_wheel lr_prefix="left" lr_reflect="1" />
     <xacro:rear_wheel lr_prefix="right" lr_reflect="-1" />
