Commit message: Gazebo launch file launches with errors

File: src/control/ros2_control/description/gazebo/qev3d.gazebo.xacro (robot description, xacro)
@@ -10,22 +10,6 @@
     <gazebo>
       <plugin filename="gz_ros2_control-system" name="gz_ros2_control::GazeboSimROS2ControlPlugin">
-        <parameters>$(find ros2_control_demo_example_9)/config/rrbot_controllers.yaml</parameters>
+        <parameters>$(find qev3d_ros2_control)/config/qev3d_controller.yaml</parameters>
       </plugin>
-    </gazebo>
-    <!-- Link1 -->
-    <gazebo reference="${prefix}base_link">
-      <material>Gazebo/Orange</material>
-    </gazebo>
-    <!-- Link2 -->
-    <gazebo reference="${prefix}link1">
-      <mu1>0.2</mu1>
-      <mu2>0.2</mu2>
-      <material>Gazebo/Yellow</material>
-    </gazebo>
-    <!-- Link3 -->
-    <gazebo reference="${prefix}link2">
-      <mu1>0.2</mu1>
-      <mu2>0.2</mu2>
-      <material>Gazebo/Orange</material>
     </gazebo>
   </xacro:macro>

File: src/operations/vehicle_urdf/urdf/qev-3d.urdf.xacro (robot description, xacro)
@@ -3,4 +3,5 @@
   xmlns:xacro="http://ros.org/wiki/xacro">
   <xacro:arg name="prefix" default="" />
+  <xacro:arg name="use_gazebo" default="false" />
   <!--  Get the parameters  -->
   <xacro:arg name="base_frame" default="base_link"/>
@@ -50,6 +51,9 @@
   </xacro:velodyne>
   <!-- ros2_control include -->
-  <!-- TODO FIXME: Fix this include path -->
-  <xacro:include filename="$(find qev3d_ros2_control)/description/qev3d.ros2_control.xacro"/>
+  <xacro:include filename="$(find qev3d_ros2_control)/ros2_control/qev3d.ros2_control.xacro"/>
   <xacro:qev3d_ros2_control name="QEV-3D" />
+  <!-- Import Gazebo definitions + plugin -->
+  <xacro:if value="$(arg use_gazebo)">
+    <xacro:include filename="$(find qev3d_ros2_control)/gazebo/qev3d.gazebo.xacro"/>
+  </xacro:if>
 </robot>

Commit message: Add materials to Gazebo model links for improved visualization

File: src/control/ros2_control/description/gazebo/qev3d.gazebo.xacro (robot description, xacro)
@@ -13,4 +13,18 @@
       </plugin>
     </gazebo>
+    <!-- Base Link -->
+    <gazebo reference="${base_frame}">
+      <material>Gazebo/Orange</material>
+    </gazebo>
+    <!-- Chassis Link -->
+    <gazebo reference="${chassis_link}">
+      <material>Gazebo/Yellow</material>
+    </gazebo>
+    <gazebo reference="virtual_rear_wheel">
+      <material>Gazebo/Orange</material>
+    </gazebo>
+    <gazebo reference="virtual_front_wheel">
+      <material>Gazebo/Orange</material>
+    </gazebo>
   </xacro:macro>
 </robot>

Commit message: Couldn't seperate link parameters to seperate files. Left TODO

File: src/control/ros2_control/description/gazebo/qev3d.gazebo.xacro (robot description, xacro)
@@ -1,10 +1,5 @@
 <?xml version="1.0"?>
-<!--
-Copied and modified from ROS1 example -
-https://github.com/ros-simulation/gazebo_ros_demos/blob/kinetic-devel/rrbot_description/urdf/rrbot.gazebo
--->
-<!-- TODO:  COPIED FROM THE EXAMPLE 9 OF ROS2_CONTROL - NEED MODIFICATION -->
 <robot xmlns:xacro="http://ros.org/wiki/xacro">
-  <xacro:macro name="qev3d_gazebo" params="prefix">
+  <xacro:macro name="qev3d_gazebo" params="prefix base_frame chassis_link">
     <!-- ros_control plugin -->
     <gazebo>
@@ -27,4 +22,20 @@
       <material>Gazebo/Orange</material>
     </gazebo>
+    <gazebo reference="left_steering_hinge">
+    </gazebo>
+    <gazebo reference="left_front_wheel">
+      <material>Gazebo/Black</material>
+    </gazebo>
+    <gazebo reference="right_steering_hinge">
+    </gazebo>
+    <gazebo reference="right_front_wheel">
+      <material>Gazebo/Red</material>
+    </gazebo>
+    <gazebo reference="left_rear_wheel">
+      <material>Gazebo/White</material>
+    </gazebo>
+    <gazebo reference="right_rear_wheel">
+      <material>Gazebo/White</material>
+    </gazebo>
   </xacro:macro>
 </robot>

File: src/operations/vehicle_urdf/urdf/vehicle.urdf.xacro (robot description, xacro)
@@ -2,4 +2,5 @@
 <robot xmlns:xacro="http://www.ros.org/wiki/xacro">
   <xacro:macro name="chassis" params="base_frame display_car">
+  <!-- TODO: collision and inertial parameters are currently placeholders. should update to match actual values OR seperate them to gazebo files if able -->
     <!-- Base Frame -->
     <link name="${base_frame}"/>

Commit message: gz_control plugin activated with gazebo launch file now. still issues with movement

File: src/control/ros2_control/description/gazebo/qev3d.gazebo.xacro (robot description, xacro)
@@ -1,5 +1,5 @@
 <?xml version="1.0"?>
 <robot xmlns:xacro="http://ros.org/wiki/xacro">
-  <xacro:macro name="qev3d_gazebo" params="prefix base_frame chassis_link">
+<xacro:macro name="qev3d_gazebo" params="prefix base_frame chassis_link">
     <!-- ros_control plugin -->
     <gazebo>
@@ -22,5 +22,7 @@
       <material>Gazebo/Orange</material>
     </gazebo>
+    <!-- Steering Hinges (if intended to be defined) -->
     <gazebo reference="left_steering_hinge">
+      <!-- Add any relevant material or other properties here -->
     </gazebo>
     <gazebo reference="left_front_wheel">
@@ -28,4 +30,5 @@
     </gazebo>
     <gazebo reference="right_steering_hinge">
+      <!-- Add any relevant material or other properties here -->
     </gazebo>
     <gazebo reference="right_front_wheel">

File: src/control/ros2_control/description/ros2_control/qev3d.ros2_control.xacro (robot description, xacro)
@@ -2,5 +2,5 @@
 <!-- Copied from the ros2 control Demo code. Change later when hardware is setup -->
 <robot xmlns:xacro="http://www.ros.org/wiki/xacro">
-  <xacro:macro name="qev3d_ros2_control" params="name use_gazebo:=^|false"> <!-- default parameters -->
+  <xacro:macro name="qev3d_ros2_control" params="name use_gazebo"> <!-- default parameters -->
     <ros2_control name="${name}" type="system">
       <hardware>

File: src/operations/vehicle_urdf/urdf/qev-3d.urdf.xacro (robot description, xacro)
@@ -48,8 +48,9 @@
   <!-- ros2_control include -->
   <xacro:include filename="$(find qev3d_ros2_control)/ros2_control/qev3d.ros2_control.xacro"/>
-  <xacro:qev3d_ros2_control name="QEV-3D" />
+  <xacro:qev3d_ros2_control name="QEV-3D" use_gazebo="$(arg use_gazebo)"/>
   <!-- Import Gazebo definitions + plugin -->
   <xacro:if value="$(arg use_gazebo)">
     <xacro:include filename="$(find qev3d_ros2_control)/gazebo/qev3d.gazebo.xacro"/>
+    <xacro:qev3d_gazebo prefix="$(arg prefix)" base_frame="$(arg base_frame)" chassis_link="chassis"/>
   </xacro:if>
 </robot>
